Commit message: gripper

File: urdf/robot.urdf (robot description, URDF)
Before this commit: robot robot, 7 links, 6 joints
Links:
- added link grasper_base_link, mass 0.22; collision box size=0.0889 0.08316 0.0889; visual mesh filename=package://talos_description/meshes/grasper_base_link.stl scale=0.001 0.001 0.001
- added link movable_claw_link, mass 0.22; collision box size=0.0635 0.07238 0.14; visual mesh filename=package://talos_description/meshes/movable_claw_link.stl scale=0.001 0.001 0.001
- added link stationary_claw_link, mass 0.22; collision box size=0.04283 0.14529 0.0862; visual mesh filename=package://talos_description/meshes/stationary_claw_link.stl scale=0.001 0.001 0.001
- added link wrist_link, mass 0.22; collision box size=0.0635 0.07238 0.14; visual mesh filename=package://talos_description/meshes/wrist_link.stl scale=0.001 0.001 0.001
- link elbow_block_link: geometry collision box size=0.06352 0.16822 0.19493; visual mesh filename=package://talos_description/meshes/elbow_block_link.stl scale=0.001 0.001 0.001
- link elbow_bracket_link: geometry collision box size=0.0651 0.151 0.2073; visual mesh filename=package://talos_description/meshes/elbow_bracket_link.stl scale=0.001 0.001 0.001
- link lower_arm_link: geometry collision box size=0.03 0.37 0.14; visual mesh filename=package://talos_description/meshes/lower_arm_link.stl scale=0.001 0.001 0.001
- link shoulder_link: geometry collision box size=0.10635 0.2 0.22; visual mesh filename=package://talos_description/meshes/shoulder_link.stl scale=0.001 0.001 0.001
- link upper_arm_link: geometry collision box size=0.02 0.55 0.15; visual mesh filename=package://talos_description/meshes/upper_arm_link.stl scale=0.001 0.001 0.001
Joints:
- added joint grasper_base_to_stationary_claw: type fixed, parent grasper_base_link, child stationary_claw_link, origin xyz=0 0.08316 0 rpy=0 0 0
- added joint lower_arm_to_wrist: type revolute, parent lower_arm_link, child wrist_link, origin xyz=0 0.289 0 rpy=0 0 0, axis 1 0 0, limit lower=-0.7853975 upper=0.7853975 effort=1000.0 velocity=1.0
- added joint stationary_claw_to_movable_claw: type revolute, parent stationary_claw_link, child movable_claw_link, origin xyz=0 0.041 0.018 rpy=0 0 0, axis 1 0 0, limit lower=-0.224399285714 upper=0.7853975 effort=1000.0 velocity=1.0
- added joint wrist_to_grasper_base: type revolute, parent wrist_link, child grasper_base_link, origin xyz=0 0.06388 0 rpy=0 0 0, axis 0 1 0, limit lower=-3.14159 upper=3.14159 effort=1000.0 velocity=1.0
