Commit message: Updated transmissions file, bug in ros control caused them to change

File: urdf/wheel/wheel.transmission.xacro (robot description, xacro)
@@ -4,7 +4,8 @@
 	    <transmission name="${prefix}_wheel_trans">
 	    <type>transmission_interface/SimpleTransmission</type>
-	    <joint name="${prefix}_wheel_joint"/>
+	    <joint name="${prefix}_wheel_joint">
+               <hardwareInterface>VelocityJointInterface</hardwareInterface>
+            </joint>
 	    <actuator name="${prefix}_wheel_motor">
-	      <hardwareInterface>VelocityJointInterface</hardwareInterface>
 	      <mechanicalReduction>1</mechanicalReduction>
 	    </actuator>
