Commit message: Added inertia and mass

File: urdf/wheel/wheel.urdf.xacro (robot description, xacro)
@@ -6,4 +6,6 @@
 	<xacro:macro name="wheel" params="prefix *origin parent">
 		<link name="${prefix}_wheel_link">
+                  <mass value="${wheel_mass}"/>
+                   <xacro:inertial_template mass="${wheel_mass}" length="${wheel_height}" width="${wheel_radius}" height="${wheel_height}"/>
 		  <visual>
 			<origin xyz="0 0 0" rpy="0 0 0"/>
@@ -25,4 +27,8 @@
                    <parent link="${parent}"/>
                    <axis xyz="0 1 0" rpy="0 0 0"/>
+                   <limit effort="100"
+                          velocity="100" />
+                   <joint_properties damping="0.0"
+                                     friction="0.0" />
                </joint>
 	</xacro:macro>

Commit message: Added wheel stls and scales

File: urdf/wheel/wheel.urdf.xacro (robot description, xacro)
@@ -11,5 +11,5 @@
 			<origin xyz="0 0 0" rpy="0 0 0"/>
 			<geometry>
-			  <cylinder length="${wheel_height*1.5}" radius="${wheel_radius}" />
+			  <mesh filename="package://talos_description/urdf/wheel/wheel.stl" scale="${scale} ${scale} ${scale}" />
 			</geometry>
 			<material name="white"/>

Commit message: Updated wheel collision sizes

File: urdf/wheel/wheel.urdf.xacro (robot description, xacro)
@@ -1,6 +1,6 @@
 <?xml version="1.0"?>
 <robot xmlns:xacro="http://www.ros.org/wiki/xacro">
-	<xacro:property name="wheel_radius" value="0.062265" />
-	<xacro:property name="wheel_height" value="0.037817" />
+	<xacro:property name="wheel_radius" value="0.0762" />
+	<xacro:property name="wheel_height" value="0.0381" />
 	<xacro:property name="wheel_mass" value="1.20" />
 	<xacro:macro name="wheel" params="prefix *origin parent">
@@ -18,5 +18,5 @@
 			<origin xyz="0 0 0" rpy="0 0 0"/>
 			<geometry>
-			  <cylinder length="${wheel_height*1.5}" radius="${wheel_radius}" />
+			  <cylinder length="${wheel_height}" radius="${wheel_radius}" />
 			</geometry>
 		  </collision>
