Commit message: Added transmission for baselink to caster_link

File: urdf/wheel/caster_wheel.transmission.xacro (robot description, xacro)
@@ -12,4 +12,13 @@
 	    </actuator>
 	  </transmission>
+           <transmission name="${prefix}_base_link_to_caster_trans">
+	    <type>transmission_interface/SimpleTransmission</type>
+	    <joint name="${prefix}_base_link_to_caster">
+               <hardwareInterface>VelocityJointInterface</hardwareInterface>
+            </joint>
+	    <actuator name="${prefix}_base_link_to_caster_motor">
+	      <mechanicalReduction>1</mechanicalReduction>
+	    </actuator>
+	  </transmission>
   </xacro:macro>
 </robot>

Commit message: Changed caster link to fixed

File: urdf/wheel/caster_wheel.transmission.xacro (robot description, xacro)
@@ -13,5 +13,5 @@
 	    </actuator>
 	  </transmission>
-           <transmission name="${prefix}_base_link_to_caster_trans">
+          <!-- <transmission name="${prefix}_base_link_to_caster_trans">
 	    <type>transmission_interface/SimpleTransmission</type>
 	    <joint name="${prefix}_base_link_to_caster">
@@ -22,5 +22,5 @@
               <hardwareInterface>JointStateInterface</hardwareInterface>
 	    </actuator>
-	  </transmission>
+	  </transmission> -->
   </xacro:macro>
 </robot>

File: urdf/wheel/caster_wheel.urdf.xacro (robot description, xacro)
@@ -49,5 +49,5 @@
 		  </collision>
 		</link>
-               <joint name="${prefix}_${parent}_to_caster" type="continuous">
+               <joint name="${prefix}_${parent}_to_caster" type="fixed">
 		   <axis xyz="0 0 1" rpy="0 0 0"/>
                    <xacro:insert_block name="origin"/>
