Commit message: lowered back wheel radius

File: urdf/wheel/back_wheel.urdf.xacro (robot description, xacro)
@@ -1,5 +1,5 @@
 <?xml version="1.0"?>
 <robot xmlns:xacro="http://www.ros.org/wiki/xacro">
-	<xacro:property name="back_wheel_radius" value="0.0762" />
+	<xacro:property name="back_wheel_radius" value="0.072805" />
 	<xacro:property name="back_wheel_height" value="0.0381" />
 	<xacro:property name="back_wheel_mass" value="1.20" />

Commit message: added caster and back wheel stls, changed wheel dimensions

File: urdf/wheel/back_wheel.urdf.xacro (robot description, xacro)
@@ -1,16 +1,16 @@
 <?xml version="1.0"?>
 <robot xmlns:xacro="http://www.ros.org/wiki/xacro">
-	<xacro:property name="back_wheel_radius" value="0.072805" />
-	<xacro:property name="back_wheel_height" value="0.0381" />
+	<xacro:property name="back_wheel_radius" value="0.0762" />
+	<xacro:property name="back_wheel_width" value="0.0127" />
 	<xacro:property name="back_wheel_mass" value="1.20" />
 	<xacro:macro name="back_wheel" params="prefix *origin parent">
 		<link name="${prefix}_back_wheel_link">
                   <mass value="${back_wheel_mass}"/>
-                   <xacro:inertial_template mass="${back_wheel_mass}" length="${back_wheel_height}" width="${back_wheel_radius}" height="${back_wheel_height}"/>
+                   <xacro:inertial_template mass="${back_wheel_mass}" length="${back_wheel_width}" width="${back_wheel_radius}" height="${back_wheel_width}"/>
 		  <visual>
-			<origin xyz="0 0 0" rpy="0 ${PI/2} 0"/>
+			<origin xyz="${-back_wheel_width/2} ${-back_wheel_radius} ${-back_wheel_radius}" rpy="0 0 0"/>
 			<geometry>
-                          <cylinder length="${back_wheel_height}" radius="${back_wheel_radius}" />
-			  <!-- <mesh filename="package://talos_description/meshes/wheel/back_wheel.stl" scale="${scale} ${scale} ${scale}" /> -->
+                          <!--<cylinder length="${back_wheel_width}" radius="${back_wheel_radius}" />-->
+			  <mesh filename="package://talos_description/meshes/wheel/back_wheel.stl" scale="${scale} ${scale} ${scale}" />
 			</geometry>
 			<material name="white"/>
@@ -19,5 +19,5 @@
                         <origin xyz="0 0 0" rpy="0 ${PI/2} 0"/>
 			<geometry>
-			  <cylinder length="${back_wheel_height}" radius="${back_wheel_radius}" />
+			  <cylinder length="${back_wheel_width}" radius="${back_wheel_radius}" />
 			</geometry>
 		  </collision>

File: urdf/wheel/caster_wheel.urdf.xacro (robot description, xacro)
@@ -2,6 +2,6 @@
 <robot xmlns:xacro="http://www.ros.org/wiki/xacro">
 	<!--need to update caster and caster wheel masses-->
-	<xacro:property name="caster_wheel_radius" value="0.0415" />
-	<xacro:property name="caster_wheel_width" value="0.02675" />
+	<xacro:property name="caster_wheel_radius" value="0.04435" />
+	<xacro:property name="caster_wheel_width" value="0.0381" />
 	<xacro:property name="caster_wheel_mass" value="1.20" />
 	<xacro:property name="caster_width" value="0.06274" />
@@ -18,8 +18,7 @@
                    <xacro:inertial_template mass="${caster_wheel_mass}" length="${caster_wheel_width}" width="${caster_wheel_radius}" height="${caster_wheel_width}"/>
 		  <visual>
-			<origin xyz="0 0 0" rpy="0 ${-PI/2} 0"/>
+			<origin xyz="0 0 0" rpy="0 0 0"/>
 			<geometry>
-			  <cylinder length="${caster_wheel_width}" radius="${caster_wheel_radius}" />
-			  <!--<mesh filename="package://talos_description/meshes/wheel/caster_wheel.stl" scale="${scale} ${scale} ${scale}" />-->
+			  <mesh filename="package://talos_description/meshes/wheel/caster_wheel.stl" scale="${scale} ${scale} ${scale}" />
 			</geometry>
 			<material name="white"/>
