Commit message: Updated

File: urdf/wheel/caster_wheel.urdf.xacro (robot description, xacro)
@@ -49,5 +49,5 @@
 		  </collision>
 		</link>
-               <joint name="${prefix}_${parent}_to_caster" type="fixed">
+               <joint name="${prefix}_${parent}_to_caster" type="continuous">
 		   <axis xyz="0 0 1" rpy="0 0 0"/>
                    <xacro:insert_block name="origin"/>

Commit message: changed friction on caster wheels so robot doesn't dance

File: urdf/wheel/caster_wheel.urdf.xacro (robot description, xacro)
@@ -58,4 +58,5 @@
                    <child link="${prefix}_caster_link"/>
                    <parent link="${parent}"/>
+		<!-- <dynamics damping="50.0" friction="50.0"/>-->
                </joint>
 		<joint name="${prefix}_caster_to_wheel" type="continuous">
@@ -66,9 +67,10 @@
 		  <child link="${prefix}_caster_wheel_link"/>
                   <parent link="${prefix}_caster_link"/>
+		  <!--<dynamics damping="50.0" friction="50.0"/>-->
 		</joint>
                 <gazebo reference="${prefix}_caster_wheel_link">
                      <!-- <selfCollide>true</selfCollide> -->
-		     <mu1 value="0.0"/>
-	             <mu2 value="0.0"/>
+		     <mu1 value="200.0"/>
+	             <mu2 value="200.0"/>
 		     <!-- <kp value="100000.0" />
 	             <kd value="1.0" /> -->
@@ -76,6 +78,6 @@
                <gazebo reference="${prefix}_caster_link">
                      <!-- <selfCollide>true</selfCollide> -->
-		     <mu1 value="0.0"/>
-	             <mu2 value="0.0"/>
+		     <mu1 value="200.0"/>
+	             <mu2 value="200.0"/>
 		     <!-- <kp value="100000.0" />
 	             <kd value="1.0" /> -->
