Commit message: Bugfix for name in trans

File: urdf/gripper/gripper.transmission.xacro (robot description, xacro)
@@ -2,8 +2,8 @@
 <robot xmlns:xacro="http://www.ros.org/wiki/xacro">
   <xacro:macro name="talos_gripper_transmission" params="prefix">
-    <transmission name="${prefix}arm_to_wrist_gripper_base_trans">
+    <transmission name="${prefix}arm_wrist_to_gripper_base_trans">
     <type>transmission_interface/SimpleTransmission</type>
-    <joint name="${prefix}arm_to_wrist_gripper_base"/>
-    <actuator name="${prefix}arm_to_wrist_gripper_base_motor">
+    <joint name="${prefix}arm_wrist_to_gripper_base"/>
+    <actuator name="${prefix}arm_wrist_to_gripper_base_motor">
       <hardwareInterface>EffortJointInterface</hardwareInterface>
       <mechanicalReduction>1</mechanicalReduction>

Commit message: Removd redundant fixed joint

File: urdf/gripper/gripper.transmission.xacro (robot description, xacro)
@@ -10,12 +10,4 @@
     </actuator>
   </transmission>
-    <transmission name="${prefix}gripper_base_to_stationary_claw_trans">
-      <type>transmission_interface/SimpleTransmission</type>
-      <joint name="${prefix}gripper_base_to_stationary_claw"/>
-      <actuator name="${prefix}gripper_base_to_stationary_claw_motor">
-        <hardwareInterface>EffortJointInterface</hardwareInterface>
-        <mechanicalReduction>1</mechanicalReduction>
-      </actuator>
-    </transmission>
     <transmission name="${prefix}gripper_stationary_claw_to_gripper_movable_claw_trans">
       <type>transmission_interface/SimpleTransmission</type>

Commit message: Updated gripper to fix transmissions as well

File: urdf/gripper/gripper.transmission.xacro (robot description, xacro)
@@ -4,7 +4,8 @@
     <transmission name="${prefix}arm_wrist_to_gripper_base_trans">
     <type>transmission_interface/SimpleTransmission</type>
-    <joint name="${prefix}arm_wrist_to_gripper_base"/>
+    <joint name="${prefix}arm_wrist_to_gripper_base">
+       <hardwareInterface>EffortJointInterface</hardwareInterface>
+    </joint>
     <actuator name="${prefix}arm_wrist_to_gripper_base_motor">
-      <hardwareInterface>EffortJointInterface</hardwareInterface>
       <mechanicalReduction>1</mechanicalReduction>
     </actuator>
@@ -12,7 +13,8 @@
     <transmission name="${prefix}gripper_stationary_claw_to_gripper_movable_claw_trans">
       <type>transmission_interface/SimpleTransmission</type>
-      <joint name="${prefix}gripper_stationary_claw_to_gripper_movable_claw"/>
+      <joint name="${prefix}gripper_stationary_claw_to_gripper_movable_claw">
+        <hardwareInterface>EffortJointInterface</hardwareInterface>
+      </joint>
       <actuator name="${prefix}gripper_stationary_claw_to_gripper_movable_claw_motor">
-        <hardwareInterface>EffortJointInterface</hardwareInterface>
         <mechanicalReduction>1</mechanicalReduction>
       </actuator>
