Commit message: Bugfix, joint had wrong name

File: urdf/arm/arm.transmission.xacro (robot description, xacro)
@@ -4,6 +4,6 @@
     <transmission name="${prefix}torso_to_arm_shoulder_trans">
     <type>transmission_interface/SimpleTransmission</type>
-    <joint name="${prefix}body_to_arm_shoulder"/>
-    <actuator name="${prefix}body_to_shoulder_motor">
+    <joint name="${prefix}torso_to_arm_shoulder"/>
+    <actuator name="${prefix}torso_to_shoulder_motor">
       <hardwareInterface>EffortJointInterface</hardwareInterface>
       <mechanicalReduction>1</mechanicalReduction>

Commit message: Fixed arm transmissions

File: urdf/arm/arm.transmission.xacro (robot description, xacro)
@@ -4,7 +4,8 @@
     <transmission name="${prefix}torso_to_arm_shoulder_trans">
     <type>transmission_interface/SimpleTransmission</type>
-    <joint name="${prefix}torso_to_arm_shoulder"/>
+    <joint name="${prefix}torso_to_arm_shoulder">
+       <hardwareInterface>EffortJointInterface</hardwareInterface>
+    </joint>
     <actuator name="${prefix}torso_to_shoulder_motor">
-      <hardwareInterface>EffortJointInterface</hardwareInterface>
       <mechanicalReduction>1</mechanicalReduction>
     </actuator>
@@ -12,7 +13,8 @@
     <transmission name="${prefix}arm_shoulder_to_arm_upper_arm_trans">
       <type>transmission_interface/SimpleTransmission</type>
-      <joint name="${prefix}arm_shoulder_to_arm_upper_arm"/>
+      <joint name="${prefix}arm_shoulder_to_arm_upper_arm">
+        <hardwareInterface>EffortJointInterface</hardwareInterface>
+      </joint>
       <actuator name="${prefix}arm_shoulder_to_arm_upper_arm_motor">
-        <hardwareInterface>EffortJointInterface</hardwareInterface>
         <mechanicalReduction>1</mechanicalReduction>
       </actuator>
@@ -20,7 +22,8 @@
     <transmission name="${prefix}arm_upper_arm_to_arm_elbow_bracket_trans">
       <type>transmission_interface/SimpleTransmission</type>
-      <joint name="${prefix}arm_upper_arm_to_arm_elbow_bracket"/>
+      <joint name="${prefix}arm_upper_arm_to_arm_elbow_bracket">
+        <hardwareInterface>EffortJointInterface</hardwareInterface>
+      </joint>
       <actuator name="${prefix}arm_upper_arm_to_arm_elbow_motor">
-        <hardwareInterface>EffortJointInterface</hardwareInterface>
         <mechanicalReduction>1</mechanicalReduction>
       </actuator>
@@ -28,7 +31,8 @@
     <transmission name="${prefix}arm_elbow_bracket_to_arm_elbow_block_trans">
       <type>transmission_interface/SimpleTransmission</type>
-      <joint name="${prefix}arm_elbow_bracket_to_arm_elbow_block"/>
+      <joint name="${prefix}arm_elbow_bracket_to_arm_elbow_block">
+           <hardwareInterface>EffortJointInterface</hardwareInterface>
+      </joint>
       <actuator name="${prefix}arm_elbow_bracket_to_arm_elbow_block_motor">
-        <hardwareInterface>EffortJointInterface</hardwareInterface>
         <mechanicalReduction>1</mechanicalReduction>
       </actuator>
@@ -36,7 +40,8 @@
     <transmission name="${prefix}arm_elbow_block_to_arm_lower_arm_trans">
       <type>transmission_interface/SimpleTransmission</type>
-      <joint name="${prefix}arm_elbow_block_to_arm_lower_arm"/>
+      <joint name="${prefix}arm_elbow_block_to_arm_lower_arm">
+        <hardwareInterface>EffortJointInterface</hardwareInterface>
+      </joint>
       <actuator name="${prefix}arm_elbow_block_to_arm_lower_arm_motor">
-        <hardwareInterface>EffortJointInterface</hardwareInterface>
         <mechanicalReduction>1</mechanicalReduction>
       </actuator>
@@ -44,7 +49,8 @@
    <transmission name="${prefix}arm_lower_arm_to_arm_wrist_trans">
       <type>transmission_interface/SimpleTransmission</type>
-      <joint name="${prefix}arm_lower_arm_to_arm_wrist"/>
+      <joint name="${prefix}arm_lower_arm_to_arm_wrist">
+        <hardwareInterface>EffortJointInterface</hardwareInterface>
+      </joint>
       <actuator name="${prefix}arm_lower_arm_to_arm_wrist_motor">
-        <hardwareInterface>EffortJointInterface</hardwareInterface>
         <mechanicalReduction>1</mechanicalReduction>
       </actuator>
