Commit message: Adjusted shoulder and torso positions

File: urdf/arm/arm.urdf.xacro (robot description, xacro)
@@ -140,6 +140,6 @@
 		 <parent link="${parent}_link" />
 		 <child link="${name}_shoulder_link" />
-		 <insert_block name="origin"/>
-		 <!--<origin xyz="${torso_width/2+shoulder_jut_offset} -${(torso_width/2)-(shoulder_slot_width/2)} ${torso_height - shoulder_height/2}" rpy="0 0 0"/>-->
+		 <!-- <xacro:insert_block name="origin"/> -->
+		  <origin xyz="${torso_width/2+shoulder_jut_offset} -${(torso_width/2)-(shoulder_slot_width/2)} ${torso_height - shoulder_height}" rpy="0 0 0"/>
 		</joint>
 		<joint name="${name}_shoulder_to_${name}_upper_arm" type="revolute">

Commit message: updated elbow bracket stl

File: urdf/arm/arm.urdf.xacro (robot description, xacro)
@@ -73,5 +73,5 @@
 		<link name="${name}_elbow_bracket_link">
 		 <visual>
-		  <origin xyz="${elbow_bracket_width/2} 0 ${-elbow_bracket_height/2}" rpy="0 0 ${PI/2}"/>
+		  <origin xyz="0 0 0" rpy="0 0 0"/>
 		  <geometry>
 			 <mesh filename="package://talos_description/meshes/arm/elbow_bracket_link.stl" scale="${scale} ${scale} ${scale}"/>

Commit message: updated shoulder stl, lower arm stl and offset

File: urdf/arm/arm.urdf.xacro (robot description, xacro)
@@ -29,5 +29,5 @@
 	<xacro:property name="lower_arm_offset" value="0.066" />
 	<xacro:property name="lower_arm_wrist_offset" value="0.015" />
-	<!--<xacro:property name="lower_arm_short_length" value="0.345" /> --><!--X Y--> <!-- theirs ours-->
+	<xacro:property name="lower_arm_short_length" value="0.28" />
 	<xacro:property name="lower_arm_width" value="0.03" /> <!--Z X-->
 	<xacro:property name="lower_arm_height" value="0.14" /> <!--Y Z-->
@@ -41,5 +41,4 @@
 		<link name="${name}_shoulder_link">
 		 <visual>
-		  <origin xyz="-${shoulder_width/2} ${-shoulder_offset} ${-shoulder_height/2}" rpy="${PI/2} 0 ${PI/2}"/>
 		  <geometry>
 			 <mesh filename="package://talos_description/meshes/arm/shoulder_link.stl" scale="${scale} ${scale} ${scale}"/>
@@ -105,5 +104,4 @@
 		<link name="${name}_lower_arm_link">
 		 <visual>
-		  <origin xyz="-${lower_arm_width/2} ${lower_arm_length-lower_arm_offset} ${lower_arm_height/2}" rpy="${-PI/2} 0 ${-PI/2}"/>
 		  <geometry>
 			 <mesh filename="package://talos_description/meshes/arm/lower_arm_link.stl" scale="${scale} ${scale} ${scale}"/>
@@ -176,5 +174,5 @@
 		 <parent link="${name}_lower_arm_link" />
 		 <child link="${name}_wrist_link" />
-		 <origin xyz="0 ${lower_arm_length-lower_arm_offset-lower_arm_wrist_offset} 0" rpy="0 0 0"/>
+		 <origin xyz="0 ${lower_arm_short_length} 0" rpy="0 0 0"/>
 		</joint>
           <xacro:talos_arm_transmission prefix=""/>

Commit message: added mimic tag to make elbow and shoulder parallel

File: urdf/arm/arm.urdf.xacro (robot description, xacro)
@@ -150,4 +150,5 @@
 		<joint name="${name}_upper_arm_to_${name}_elbow_bracket" type="revolute">
 		 <limit velocity="1.0" effort="1000.0" lower="${-PI/4}" upper="${PI/4}"/>
+		 <mimic joint="${name}_shoulder_to_${name}_upper_arm" multiplier="-1" />
 		 <axis xyz="1 0 0"/>
 		 <parent link="${name}_upper_arm_link" />

Commit message: added mimic plugin for arm

File: urdf/arm/arm.urdf.xacro (robot description, xacro)
@@ -150,5 +150,5 @@
 		<joint name="${name}_upper_arm_to_${name}_elbow_bracket" type="revolute">
 		 <limit velocity="1.0" effort="1000.0" lower="${-PI/4}" upper="${PI/4}"/>
-		 <mimic joint="${name}_shoulder_to_${name}_upper_arm" multiplier="-1" />
+		 <!--<mimic joint="${name}_shoulder_to_${name}_upper_arm" multiplier="-1" />-->
 		 <axis xyz="1 0 0"/>
 		 <parent link="${name}_upper_arm_link" />
@@ -177,4 +177,11 @@
 		 <origin xyz="0 ${lower_arm_short_length} 0" rpy="0 0 0"/>
 		</joint>
+             <gazebo>
+	       <plugin name="mimic_plugin" filename="libtalos_description.so">
+                <joint>${name}_upper_arm_to_${name}_elbow_bracket</joint>
+                <mimicJoint>${name}_shoulder_to_${name}_upper_arm</mimicJoint>
+                <multiplier>-1.0</multiplier>
+               </plugin>
+              </gazebo>
           <xacro:talos_arm_transmission prefix=""/>
 	</xacro:macro>
