Commit message: Updated torso transmissions

File: urdf/torso/torso.transmission.xacro (robot description, xacro)
@@ -4,7 +4,8 @@
     <transmission name="${prefix}base_to_torso_trans">
     <type>transmission_interface/SimpleTransmission</type>
-    <joint name="${prefix}base_to_torso"/>
+    <joint name="${prefix}base_to_torso">
+      <hardwareInterface>EffortJointInterface</hardwareInterface>
+    </joint>
     <actuator name="${prefix}base_to_torso_motor">
-      <hardwareInterface>EffortJointInterface</hardwareInterface>
       <mechanicalReduction>1</mechanicalReduction>
     </actuator>
