Commit message: Added wheels and positioned them correctly

File: robot/robot.gazebo.xacro (robot description, xacro)
@@ -9,18 +9,5 @@
 	<xacro:include filename="$(find talos_description)/urdf/arm/arm.urdf.xacro" />
 	<xacro:include filename="$(find talos_description)/urdf/gripper/gripper.urdf.xacro" />
-        <xacro:include filename="$(find talos_description)/urdf/wheel/wheel.urdf.xacro" />
 	<xacro:base name="base"/>
-        <xacro:wheel prefix="fl" parent="base_link">
-           <origin xyz="0 0 0" rpy="0 0 0"/>
-        </xacro:wheel>
-        <xacro:wheel prefix="fr" parent="base_link">
-           <origin xyz="0 0 0" rpy="0 0 0"/>
-        </xacro:wheel>
-        <xacro:wheel prefix="bl" parent="base_link">
-           <origin xyz="0 0 0" rpy="0 0 0"/>
-        </xacro:wheel>
-        <xacro:wheel prefix="br" parent="base_link">
-           <origin xyz="0 0 0" rpy="0 0 0"/>
-        </xacro:wheel>
 	<xacro:torso name="torso" parent="base">
 		<origin xyz="0 0 ${base_height}" rpy="0 0 0"/>

File: robot/robot.urdf.xacro (robot description, xacro)
@@ -9,18 +9,5 @@
 	<xacro:include filename="$(find talos_description)/urdf/arm/arm.urdf.xacro" />
 	<xacro:include filename="$(find talos_description)/urdf/gripper/gripper.urdf.xacro" />
-        <xacro:include filename="$(find talos_description)/urdf/wheel/wheel.urdf.xacro" />
 	<xacro:base name="base"/>
-        <xacro:wheel prefix="fl" parent="base_link">
-           <origin xyz="0 0 0" rpy="0 0 0"/>
-        </xacro:wheel>
-        <xacro:wheel prefix="fr" parent="base_link">
-           <origin xyz="0 0 0" rpy="0 0 0"/>
-        </xacro:wheel>
-        <xacro:wheel prefix="bl" parent="base_link">
-           <origin xyz="0 0 0" rpy="0 0 0"/>
-        </xacro:wheel>
-        <xacro:wheel prefix="br" parent="base_link">
-           <origin xyz="0 0 0" rpy="0 0 0"/>
-        </xacro:wheel>
 	<xacro:torso name="torso" parent="base">
 		<origin xyz="0 0 ${base_height}" rpy="0 0 0"/>

File: urdf/base/base.urdf.xacro (robot description, xacro)
@@ -1,4 +1,5 @@
 <?xml version="1.0"?>
 <robot xmlns:xacro="http://www.ros.org/wiki/xacro">
+        <xacro:include filename="$(find talos_description)/urdf/wheel/wheel.urdf.xacro" />
 	<xacro:property name="base_width" value="0.62265" />
 	<xacro:property name="base_height" value="0.37817" />
@@ -21,4 +22,16 @@
 		  <xacro:inertial_template mass="${base_mass}" length="${base_width}" width="${base_width}" height="${base_height}"/>
 		</link>
+                <xacro:wheel prefix="fl" parent="base_link">
+                    <origin xyz="${base_width/3} ${base_width/3} 0" rpy="0 ${PI/2} 0"/>
+                </xacro:wheel>
+                <xacro:wheel prefix="fr" parent="base_link">
+                    <origin xyz="${-base_width/3} ${base_width/3} 0" rpy="0 ${PI/2} 0"/>
+                </xacro:wheel>
+                <xacro:wheel prefix="bl" parent="base_link">
+                    <origin xyz="${base_width/3} ${-base_width/3} 0" rpy="0 ${PI/2} 0"/>
+                </xacro:wheel>
+                <xacro:wheel prefix="br" parent="base_link">
+                   <origin xyz="${-base_width/3} ${-base_width/3} 0" rpy="0 ${PI/2} 0"/>
+                </xacro:wheel>
 	</xacro:macro>
 </robot>

Commit message: wheels still not working

File: robot/robot.gazebo.xacro (robot description, xacro)
@@ -52,14 +52,14 @@
     </gazebo>
     <gazebo reference="bl_wheel_link">
-           <selfCollide>true</selfCollide>
+           <selfCollide>false</selfCollide>
     </gazebo>
     <gazebo reference="br_wheel_link">
-           <selfCollide>true</selfCollide>
+           <selfCollide>false</selfCollide>
     </gazebo>
      <gazebo reference="fl_wheel_link">
-           <selfCollide>true</selfCollide>
+           <selfCollide>false</selfCollide>
     </gazebo>
      <gazebo reference="fr_wheel_link">
-           <selfCollide>true</selfCollide>
+           <selfCollide>false</selfCollide>
     </gazebo>
 </robot>

File: urdf/base/base.urdf.xacro (robot description, xacro)
@@ -24,14 +24,14 @@
 		</link>
                 <xacro:wheel prefix="fl" parent="base_link">
-                    <origin xyz="${base_width/3} ${base_width/3} 0" rpy="0 ${PI/2} ${PI/2}"/>
+                    <origin xyz="${base_width/3} ${base_width/3} 0" rpy="0 ${PI/2} 0"/>
                 </xacro:wheel>
                 <xacro:wheel prefix="fr" parent="base_link">
-                    <origin xyz="${-base_width/3} ${base_width/3} 0" rpy="0 ${PI/2} ${PI/2}"/>
+                    <origin xyz="${-base_width/3} ${base_width/3} 0" rpy="0 ${PI/2} 0"/>
                 </xacro:wheel>
                 <xacro:wheel prefix="bl" parent="base_link">
-                    <origin xyz="${base_width/3} ${-base_width/3} 0" rpy="0 ${PI/2} ${PI/2}"/>
+                    <origin xyz="${base_width/3} ${-base_width/3} 0" rpy="0 ${PI/2} 0"/>
                 </xacro:wheel>
                 <xacro:wheel prefix="br" parent="base_link">
-                   <origin xyz="${-base_width/3} ${-base_width/3} 0" rpy="0 ${PI/2} ${PI/2}"/>
+                   <origin xyz="${-base_width/3} ${-base_width/3} 0" rpy="0 ${PI/2} 0"/>
                 </xacro:wheel>
 		<xacro:talos_wheel_transmission prefix="bl"/>

File: urdf/wheel/wheel.urdf.xacro (robot description, xacro)
@@ -11,5 +11,6 @@
 			<origin xyz="0 0 0" rpy="0 0 0"/>
 			<geometry>
-			  <mesh filename="package://talos_description/urdf/wheel/wheel.stl" scale="${scale} ${scale} ${scale}" />
+                          <cylinder length="${wheel_height}" radius="${wheel_radius}" />
+			  <!-- <mesh filename="package://talos_description/urdf/wheel/wheel.stl" scale="${scale} ${scale} ${scale}" /> -->
 			</geometry>
 			<material name="white"/>
@@ -33,8 +34,8 @@
                </joint>
                <gazebo reference="${prefix}_wheel_link">
-		     <mu1 value="1.0"/>
-	              <mu2 value="1.0"/>
-		     <kp value="10000000.0" />
-	             <kd value="1.0" />
+		     <!-- <mu1 value="1.0"/>
+	             <mu2 value="1.0"/>
+		     <kp value="100000.0" />
+	             <kd value="1.0" /> -->
 	             <fdir1 value="1 0 0"/>
 	       </gazebo>

Commit message: Updated urdf

File: robot/robot.gazebo.xacro (robot description, xacro)
@@ -51,15 +51,3 @@
            <selfCollide>true</selfCollide>
     </gazebo>
-    <gazebo reference="bl_wheel_link">
-           <selfCollide>false</selfCollide>
-    </gazebo>
-    <gazebo reference="br_wheel_link">
-           <selfCollide>false</selfCollide>
-    </gazebo>
-     <gazebo reference="fl_wheel_link">
-           <selfCollide>false</selfCollide>
-    </gazebo>
-     <gazebo reference="fr_wheel_link">
-           <selfCollide>false</selfCollide>
-    </gazebo>
 </robot>

File: urdf/base/base.urdf.xacro (robot description, xacro)
@@ -24,14 +24,14 @@
 		</link>
                 <xacro:wheel prefix="fl" parent="base_link">
-                    <origin xyz="${base_width/3} ${base_width/3} 0" rpy="0 ${PI/2} 0"/>
+                    <origin xyz="${base_width/3} ${base_width/3} 0" rpy="0 ${PI/2} ${PI/2}"/>
                 </xacro:wheel>
                 <xacro:wheel prefix="fr" parent="base_link">
-                    <origin xyz="${-base_width/3} ${base_width/3} 0" rpy="0 ${PI/2} 0"/>
+                    <origin xyz="${-base_width/3} ${base_width/3} 0" rpy="0 ${PI/2} ${PI/2}"/>
                 </xacro:wheel>
                 <xacro:wheel prefix="bl" parent="base_link">
-                    <origin xyz="${base_width/3} ${-base_width/3} 0" rpy="0 ${PI/2} 0"/>
+                    <origin xyz="${base_width/3} ${-base_width/3} 0" rpy="0 ${PI/2} ${PI/2}"/>
                 </xacro:wheel>
                 <xacro:wheel prefix="br" parent="base_link">
-                   <origin xyz="${-base_width/3} ${-base_width/3} 0" rpy="0 ${PI/2} 0"/>
+                   <origin xyz="${-base_width/3} ${-base_width/3} 0" rpy="0 ${PI/2} ${PI/2}"/>
                 </xacro:wheel>
 		<xacro:talos_wheel_transmission prefix="bl"/>

File: urdf/wheel/wheel.urdf.xacro (robot description, xacro)
@@ -17,5 +17,5 @@
 		  </visual>
 		  <collision>
-			<origin xyz="0 0 0" rpy="0 0 0"/>
+                        <origin xyz="0 0 0" rpy="0 0 0"/>
 			<geometry>
 			  <cylinder length="${wheel_height}" radius="${wheel_radius}" />
@@ -34,9 +34,10 @@
                </joint>
                <gazebo reference="${prefix}_wheel_link">
+                     <selfCollide>true</selfCollide>
 		     <!-- <mu1 value="1.0"/>
 	             <mu2 value="1.0"/>
 		     <kp value="100000.0" />
 	             <kd value="1.0" /> -->
-	             <fdir1 value="1 0 0"/>
+	             <!-- <fdir1 value="1 0 0"/> -->
 	       </gazebo>
 	</xacro:macro>

Commit message: Added skeleton head to model

File: robot/robot.gazebo.xacro (robot description, xacro)
@@ -9,4 +9,5 @@
 	<xacro:include filename="$(find talos_description)/urdf/arm/arm.urdf.xacro" />
 	<xacro:include filename="$(find talos_description)/urdf/gripper/gripper.urdf.xacro" />
+        <xacro:include filename="$(find talos_description)/urdf/head/head.urdf.xacro" />
 	<xacro:base name="base"/>
 	<xacro:torso name="torso" parent="base">
@@ -19,4 +20,7 @@
 		<origin xyz="0 ${wrist_length - wrist_offset} 0" rpy="0 0 0"/>
 	</xacro:gripper>
+        <xacro:head prefix="" parent="torso_link">
+                <origin xyz="0 0 0" rpy="0 0 0"/>
+        </xacro:head>
        <gazebo>
           <plugin name="gazebo_ros_control" filename="libgazebo_ros_control.so">

File: urdf/head/head.urdf.xacro (robot description, xacro)
@@ -67,4 +67,5 @@
                      <selfCollide>true</selfCollide>
 	       </gazebo>
+         <xacro:include filename="$(find talos_description)/urdf/head/head.transmission.xacro" />
 	</xacro:macro>
 </robot>

Commit message: Added neck position to talos

File: robot/robot.gazebo.xacro (robot description, xacro)
@@ -21,5 +21,5 @@
 	</xacro:gripper>
         <xacro:head prefix="" parent="torso_link">
-                <origin xyz="0 0 0" rpy="0 0 0"/>
+                <origin xyz="0 0 ${torso_height - head_offset}" rpy="${PI/2} 0 ${PI}"/>
         </xacro:head>
        <gazebo>

File: urdf/head/head.urdf.xacro (robot description, xacro)
@@ -2,4 +2,5 @@
 <robot xmlns:xacro="http://www.ros.org/wiki/xacro">
 	<xacro:property name="head_mass" value="0.20" />
+        <xacro:property name="head_offset" value="0.085" />
          <xacro:include filename="$(find talos_description)/urdf/head/head.transmission.xacro" />
 	<xacro:macro name="head" params="prefix parent *origin">

Commit message: updated head pose temporarily until new joint position stls are in

File: robot/robot.gazebo.xacro (robot description, xacro)
@@ -21,5 +21,5 @@
 	</xacro:gripper>
         <xacro:head prefix="" parent="torso_link">
-                <origin xyz="0 0 ${torso_height - head_offset}" rpy="${PI/2} 0 ${PI}"/>
+                <origin xyz="0 0 ${torso_height -neck_offset}" rpy="${PI/2} 0 ${PI}"/>
         </xacro:head>
        <gazebo>

File: urdf/head/head.urdf.xacro (robot description, xacro)
@@ -2,5 +2,7 @@
 <robot xmlns:xacro="http://www.ros.org/wiki/xacro">
 	<xacro:property name="head_mass" value="0.20" />
-        <xacro:property name="head_offset" value="0.085" />
+        <xacro:property name="neck_offset" value="0.085" />
+        <xacro:property name="head_offset" value="0.075" />
+        <xacro:property name="neck_alignment" value="${PI/12}" />
          <xacro:include filename="$(find talos_description)/urdf/head/head.transmission.xacro" />
 	<xacro:macro name="head" params="prefix parent *origin">
@@ -10,5 +12,5 @@
                    <xacro:inertial_template mass="${head_mass}" length="${head_mass}" width="${head_mass}" height="${head_mass}"/>
 		  <visual>
-			<origin xyz="0 0 0" rpy="0 0 0"/>
+			<origin xyz="0 ${head_offset} 0" rpy="0 0 0"/>
 			<geometry>
                            <mesh filename="package://talos_description/urdf/head/head.stl" scale="${scale} ${scale} ${scale}" />
@@ -28,5 +30,5 @@
                    <xacro:inertial_template mass="${head_mass}" length="${head_mass}" width="${head_mass}" height="${head_mass}"/>
 		  <visual>
-			<origin xyz="0 0 0" rpy="0 0 0"/>
+			<origin xyz="0 0 0" rpy="0 -${neck_alignment} 0"/>
 			<geometry>
                            <mesh filename="package://talos_description/urdf/head/neck.stl" scale="${scale} ${scale} ${scale}" />

Commit message: more stable teleop

File: robot/robot.gazebo.xacro (robot description, xacro)
@@ -12,5 +12,5 @@
 	<xacro:base name="base"/>
 	<xacro:torso name="torso" parent="base">
-		<origin xyz="0 0 ${base_height}" rpy="0 0 0"/>
+		<origin xyz="0 0 ${base_height}" rpy="0 0 ${PI}"/>
 	</xacro:torso>
 	<xacro:arm name="arm" parent="torso">

File: urdf/wheel/back_wheel.urdf.xacro (robot description, xacro)
@@ -35,8 +35,8 @@
                <gazebo reference="${prefix}_back_wheel_link">
                      <selfCollide>true</selfCollide>
-		  <!--   <mu1 value="1.0"/>
-	             <mu2 value="1.0"/>
-		     <kp value="100000.0" />
-	             <kd value="1.0" /> -->
+		     <mu1 value="50.0"/>
+	             <mu2 value="50.0"/>
+		    <!-- <kp value="100000.0" />
+	             <kd value="1.0" />-->
 	             <!-- <fdir1 value="1 0 0"/> -->
 	       </gazebo>

File: urdf/wheel/caster_wheel.urdf.xacro (robot description, xacro)
@@ -63,11 +63,11 @@
                   <parent link="${prefix}_caster_link"/>
 		</joint>
-               <!-- <gazebo reference="${prefix}_caster_wheel_link">
-                     <selfCollide>true</selfCollide>
-		     <mu1 value="1.0"/>
-	             <mu2 value="1.0"/>
-		     <kp value="100000.0" />
-	             <kd value="1.0" />
-	       </gazebo> -->
+                <gazebo reference="${prefix}_caster_wheel_link">
+                     <!-- <selfCollide>true</selfCollide> -->
+		     <mu1 value="50.0"/>
+	             <mu2 value="50.0"/>
+		     <!-- <kp value="100000.0" />
+	             <kd value="1.0" /> -->
+	       </gazebo>
 	</xacro:macro>
 </robot>
