Commit message: Fixed minor urdf bug

File: robot/robot.urdf (robot description, URDF)
Before this commit: robot talos, 11 links, 10 joints
Links:
- added link bl_wheel_link; collision cylinder length=0.037817 radius=0.062265; visual cylinder length=0.037817 radius=0.062265
- added link br_wheel_link; collision cylinder length=0.037817 radius=0.062265; visual cylinder length=0.037817 radius=0.062265
- added link fl_wheel_link; collision cylinder length=0.037817 radius=0.062265; visual cylinder length=0.037817 radius=0.062265
- added link fr_wheel_link; collision cylinder length=0.037817 radius=0.062265; visual cylinder length=0.037817 radius=0.062265
Joints:
- added joint bl_wheel_joint: type continuous, parent base_link, child bl_wheel_link, origin xyz=0 0 0 rpy=0 0 0, axis 0 1 0
- added joint br_wheel_joint: type continuous, parent base_link, child br_wheel_link, origin xyz=0 0 0 rpy=0 0 0, axis 0 1 0
- added joint fl_wheel_joint: type continuous, parent base_link, child fl_wheel_link, origin xyz=0 0 0 rpy=0 0 0, axis 0 1 0
- added joint fr_wheel_joint: type continuous, parent base_link, child fr_wheel_link, origin xyz=0 0 0 rpy=0 0 0, axis 0 1 0

File: urdf/wheel/wheel.urdf.xacro (robot description, xacro)
@@ -19,5 +19,4 @@
 			</geometry>
 		  </collision>
-		 <!-- <xacro:inertial_template mass="${base_mass}" length="${base_width}" width="${base_width}" height="${base_height}"/> -->
 		</link>
                <joint name="${prefix}_wheel_joint" type="continuous">

Commit message: Updated physical model and rviz model

File: robot/robot.urdf (robot description, URDF)
Before this commit: robot talos, 15 links, 14 joints
Links:
- removed link bl_wheel_link
- removed link br_wheel_link
- removed link fl_wheel_link
- removed link fr_wheel_link
- added link bl_back_wheel_link, mass 1.2; collision cylinder length=0.0381 radius=0.072805; visual cylinder length=0.0381 radius=0.072805
- added link br_back_wheel_link, mass 1.2; collision cylinder length=0.0381 radius=0.072805; visual cylinder length=0.0381 radius=0.072805
- added link fl_caster_link, mass 1.2; collision box size=0.06274 0.07339 0.12223; visual mesh filename=package://talos_description/meshes/wheel/caster.stl scale=0.001 0.001 0.001
- added link fl_caster_wheel_link, mass 1.2; collision cylinder length=0.02675 radius=0.0415; visual cylinder length=0.02675 radius=0.0415
- added link fr_caster_link, mass 1.2; collision box size=0.06274 0.07339 0.12223; visual mesh filename=package://talos_description/meshes/wheel/caster.stl scale=0.001 0.001 0.001
- added link fr_caster_wheel_link, mass 1.2; collision cylinder length=0.02675 radius=0.0415; visual cylinder length=0.02675 radius=0.0415
- added link talos_head_link, mass 0.2; collision mesh filename=package://talos_description/urdf/head/head.stl scale=0.001 0.001 0.001; visual mesh filename=package://talos_description/urdf/head/head.stl scale=0.001 0.001 0.001
- added link talos_neck_link, mass 0.2; collision mesh filename=package://talos_description/urdf/head/neck.stl scale=0.001 0.001 0.001; visual mesh filename=package://talos_description/urdf/head/neck.stl scale=0.001 0.001 0.001
- link base_link: geometry collision box size=0.62265 0.62265 0.37817; visual mesh filename=package://talos_description/meshes/base/base_link.stl scale=0.001 0.001 0.001
- link gripper_base_link: geometry collision cylinder length=0.08316 radius=0.04445; visual mesh filename=package://talos_description/meshes/gripper/gripper_base_lin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 scale=0.001 0.001 0.001
- link gripper_movable_claw_link: geometry collision mesh filename=package://talos_description/meshes/gripper/movable_claw_lin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 scale=0.001 0.001 0.001; visual mesh filename=package://talos_description/meshes/gripper/movable_claw_lin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 scale=0.001 0.001 0.001
- link gripper_stationary_claw_link: geometry collision mesh filename=package://talos_description/meshes/gripper/stationary_claw_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 scale=0.001 0.001 0.001; visual mesh filename=package://talos_description/meshes/gripper/stationary_claw_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 scale=0.001 0.001 0.001
- link torso_link: geometry collision box size=0.4324 0.4324 1.03818; visual mesh filename=package://talos_description/meshes/torso/torso_link.stl scale=0.001 0.001 0.001
Joints:
- removed joint bl_wheel_joint
- removed joint br_wheel_joint
- removed joint fl_wheel_joint
- removed joint fr_wheel_joint
- added joint bl_back_wheel_joint: type continuous, parent base_link, child bl_back_wheel_link, origin xyz=0.229125 -0.2 -0.040132 rpy=0 0 0, axis 1 0 0, limit effort=100 velocity=100
- added joint br_back_wheel_joint: type continuous, parent base_link, child br_back_wheel_link, origin xyz=-0.229125 -0.2 -0.040132 rpy=0 0 0, axis 1 0 0, limit effort=100 velocity=100
- added joint fl_base_link_to_caster: type continuous, parent base_link, child fl_caster_link, origin xyz=0.2175 0.21745 0 rpy=0 0 0, axis 0 0 1
- added joint fl_caster_to_wheel: type continuous, parent fl_caster_link, child fl_caster_wheel_link, origin xyz=0 -0.0293624 -0.071437 rpy=0 0 0, axis 1 0 0, limit effort=100 velocity=100
- added joint fr_base_link_to_caster: type continuous, parent base_link, child fr_caster_link, origin xyz=-0.2175 0.21745 0 rpy=0 0 0, axis 0 0 1
- added joint fr_caster_to_wheel: type continuous, parent fr_caster_link, child fr_caster_wheel_link, origin xyz=0 -0.0293624 -0.071437 rpy=0 0 0, axis 1 0 0, limit effort=100 velocity=100
- added joint talos_head_joint: type fixed, parent talos_neck_link, child talos_head_link, origin xyz=0 0 0 rpy=0 0 0, axis 0 1 0
- added joint talos_neck_joint: type fixed, parent torso_link, child talos_neck_link, origin xyz=0 0 0.95318 rpy=1.57079632679 0 3.14159265359, axis 0 1 0
- joint arm_shoulder_to_arm_upper_arm: origin xyz=0.053175 0.095 0 rpy=0 0 0 -> xyz=0 0.095 0 rpy=0 0 0
- joint base_to_torso: origin xyz=0 0 0.37817 rpy=0 0 0 -> xyz=0 0 0.37817 rpy=0 0 3.14159265359
- joint torso_to_arm_shoulder: origin xyz=0.2162 0 0.89318 rpy=0 0 0 -> xyz=0.276375 -0.1517 0.81818 rpy=0 0 0

File: robot/robot.urdf.xacro (robot description, xacro)
@@ -9,13 +9,17 @@
 	<xacro:include filename="$(find talos_description)/urdf/arm/arm.urdf.xacro" />
 	<xacro:include filename="$(find talos_description)/urdf/gripper/gripper.urdf.xacro" />
+        <xacro:include filename="$(find talos_description)/urdf/head/head.urdf.xacro" />
 	<xacro:base name="base"/>
 	<xacro:torso name="torso" parent="base">
-		<origin xyz="0 0 ${base_height-base_skirt_height_guestimate}" rpy="0 0 0"/>
+		<origin xyz="0 0 ${base_height}" rpy="0 0 ${PI}"/>
 	</xacro:torso>
 	<xacro:arm name="arm" parent="torso">
-		<origin xyz="${torso_width/2+shoulder_jut_offset} -${(torso_width/2)-(shoulder_slot_width/2)} ${torso_height - shoulder_height/2}" rpy="0 0 0"/>
+		<origin xyz="${torso_width/2} 0 ${torso_height - shoulder_height/2}" rpy="0 0 0"/>
 	</xacro:arm>
 	<xacro:gripper name="gripper" parent="arm">
 		<origin xyz="0 ${wrist_length - wrist_offset} 0" rpy="0 0 0"/>
 	</xacro:gripper>
+        <xacro:head prefix="" parent="torso_link">
+                <origin xyz="0 0 ${torso_height -neck_offset}" rpy="${PI/2} 0 ${PI}"/>
+        </xacro:head>
 </robot>
