Commit message: Added wheel macros into robot.urdf.xacro

File: robot/robot.urdf.xacro (robot description, xacro)
@@ -9,5 +9,18 @@
 	<xacro:include filename="$(find talos_description)/urdf/arm/arm.urdf.xacro" />
 	<xacro:include filename="$(find talos_description)/urdf/gripper/gripper.urdf.xacro" />
+        <xacro:include filename="$(find talos_description)/urdf/wheel/wheel.urdf.xacro" />
 	<xacro:base name="base"/>
+        <xacro:wheel prefix="fl" parent="base_link">
+           <origin xyz="0 0 0" rpy="0 0 0"/>
+        </xacro:wheel>
+        <xacro:wheel prefix="fr" parent="base_link">
+           <origin xyz="0 0 0" rpy="0 0 0"/>
+        </xacro:wheel>
+        <xacro:wheel prefix="bl" parent="base_link">
+           <origin xyz="0 0 0" rpy="0 0 0"/>
+        </xacro:wheel>
+        <xacro:wheel prefix="br" parent="base_link">
+           <origin xyz="0 0 0" rpy="0 0 0"/>
+        </xacro:wheel>
 	<xacro:torso name="torso" parent="base">
 		<origin xyz="0 0 ${base_height}" rpy="0 0 0"/>

Commit message: updated torso stl, repositioned shoulder joint

File: robot/robot.urdf.xacro (robot description, xacro)
@@ -14,5 +14,5 @@
 	</xacro:torso>
 	<xacro:arm name="arm" parent="torso">
-		<origin xyz="${torso_width/2} 0 ${torso_height - shoulder_height/2}" rpy="0 0 0"/>
+		<origin xyz="${torso_width/2+shoulder_jut_offset} -${(torso_width/2)-(shoulder_slot_width/2)} ${torso_height - shoulder_height/2}" rpy="0 0 0"/>
 	</xacro:arm>
 	<xacro:gripper name="gripper" parent="arm">

File: urdf/arm/arm.urdf.xacro (robot description, xacro)
@@ -5,7 +5,9 @@
 	<xacro:property name="shoulder_short_length" value="0.095" />
 	<xacro:property name="shoulder_offset" value="0.035" />
+	<xacro:property name="shoulder_jut_offset" value= "0.060175" />
 	<xacro:property name="shoulder_width" value="0.10635" />
 	<xacro:property name="shoulder_height" value="0.22" />
 	<xacro:property name="shoulder_mass" value="0.22" />
+	<xacro:property name="shoulder_slot_width" value="0.129" />
 	<xacro:property name="upper_arm_length" value="0.55" />
 	<xacro:property name="upper_arm_short_length" value="0.4" />
@@ -39,5 +41,5 @@
 		<link name="${name}_shoulder_link">
 		 <visual>
-		  <origin xyz="0 ${-shoulder_offset} ${-shoulder_height/2}" rpy="${PI/2} 0 ${PI/2}"/>
+		  <origin xyz="-${shoulder_width/2} ${-shoulder_offset} ${-shoulder_height/2}" rpy="${PI/2} 0 ${PI/2}"/>
 		  <geometry>
 			 <mesh filename="package://talos_description/meshes/arm/shoulder_link.stl" scale="${scale} ${scale} ${scale}"/>
@@ -139,5 +141,5 @@
 		 <child link="${name}_shoulder_link" />
 		 <insert_block name="origin"/>
-		 <!--<origin xyz="${body_width/2} 0 ${body_height - shoulder_height/2}" rpy="0 0 0"/>-->
+		 <!--<origin xyz="${torso_width/2+shoulder_jut_offset} -${(torso_width/2)-(shoulder_slot_width/2)} ${torso_height - shoulder_height/2}" rpy="0 0 0"/>-->
 		</joint>
 		<joint name="${name}_shoulder_to_${name}_upper_arm" type="revolute">
@@ -146,5 +148,5 @@
 		 <parent link="${name}_shoulder_link" />
 		 <child link="${name}_upper_arm_link" />
-		 <origin xyz="${shoulder_width/2} ${shoulder_short_length} 0" rpy="0 0 0"/>
+		 <origin xyz="0 ${shoulder_short_length} 0" rpy="0 0 0"/>
 		</joint>
 		<joint name="${name}_upper_arm_to_${name}_elbow_bracket" type="revolute">

File: urdf/torso/torso.urdf.xacro (robot description, xacro)
@@ -2,13 +2,15 @@
 <robot xmlns:xacro="http://www.ros.org/wiki/xacro">
 	<xacro:property name="torso_width" value="0.4324" />
-	<xacro:property name="torso_height" value="1.00318" />
+	<xacro:property name="torso_height" value="1.03818" />
 	<xacro:property name="torso_mass" value="5.20" />
+	<xacro:property name="torso_offset" value="0.23965" />
         <xacro:include filename="$(find talos_description)/urdf/torso/torso.transmission.xacro"/>
 	<xacro:macro name="torso" params="name parent *origin">
 		<link name="${name}_link">
 		 <visual>
-		  <origin xyz="0 0 ${torso_height/2}" rpy="0 0 0"/>
+		  <origin xyz="-${torso_width/2} ${torso_width/2} -${torso_offset}" rpy="0 0 -${PI/2}"/>
 		  <geometry>
-			 <box size="${torso_width} ${torso_width} ${torso_height}" />
+			 <!--<box size="${torso_width} ${torso_width} ${torso_height}" />-->
+<mesh filename="package://talos_description/meshes/torso/torso_link.stl" scale="${scale} ${scale} ${scale}"/>
 		  </geometry>
 		  <material name="white"/>

Commit message: added detailed base

File: robot/robot.urdf.xacro (robot description, xacro)
@@ -11,5 +11,5 @@
 	<xacro:base name="base"/>
 	<xacro:torso name="torso" parent="base">
-		<origin xyz="0 0 ${base_height}" rpy="0 0 0"/>
+		<origin xyz="0 0 ${base_height-base_skirt_height_guestimate}" rpy="0 0 0"/>
 	</xacro:torso>
 	<xacro:arm name="arm" parent="torso">

File: urdf/base/base.urdf.xacro (robot description, xacro)
@@ -5,11 +5,12 @@
 	<xacro:property name="base_width" value="0.62265" />
 	<xacro:property name="base_height" value="0.37817" />
+	<xacro:property name="base_skirt_height_guestimate" value="0.073" />
 	<xacro:property name="base_mass" value="8.20" />
 	<xacro:macro name="base" params="name">
 		<link name="${name}_link">
 		  <visual>
-			<origin xyz="0 0 ${base_height/2}" rpy="0 0 0"/>
+			<origin xyz="${base_width/2} ${base_width/2} 0" rpy="0 0 ${PI}"/>
 			<geometry>
-			  <box size="${base_width} ${base_width} ${base_height}" />
+			  <mesh filename="package://talos_description/meshes/base/base_link.stl" scale="${scale} ${scale} ${scale}"/>
 			</geometry>
 			<material name="white"/>

Commit message: neck pan has correct angle

File: robot/robot.urdf.xacro (robot description, xacro)
@@ -22,5 +22,5 @@
 	</xacro:gripper>
         <xacro:head prefix="" parent="torso_link">
-                <origin xyz="0 0 ${torso_height -neck_offset}" rpy="${PI/2} 0 ${PI}"/>
+                <origin xyz="0 0 ${torso_height -neck_offset}" rpy="${PI/2} 0 0"/>
         </xacro:head>
         <!-- Add sensors to talos -->

File: urdf/head/head.urdf.xacro (robot description, xacro)
@@ -5,4 +5,5 @@
         <xacro:property name="head_offset" value="0.075" />
         <xacro:property name="neck_alignment" value="${PI/12}" />
+        <xacro:property name="pan_rotation_alignment" value="${PI/8}"/>
         <xacro:include filename="$(find talos_description)/urdf/head/head.transmission.xacro" />
 	<xacro:macro name="head" params="prefix parent *origin">
@@ -30,5 +31,5 @@
                    <xacro:inertial_template mass="${head_mass}" length="${head_mass/12}" width="${head_mass/12}" height="${head_mass/12}"/>
 		  <visual>
-			<origin xyz="0 0 0" rpy="0 -${neck_alignment} 0"/>
+			<origin xyz="0 0 0" rpy="0 ${PI/4} 0"/>
 			<geometry>
                            <mesh filename="package://talos_description/meshes/head/pan_neck.stl" scale="${scale} ${scale} ${scale}" />
@@ -78,5 +79,5 @@
                    <child link="${prefix}talos_stationary_neck_link"/>
                    <parent link="${parent}"/>
-                   <axis xyz="0 1 0" rpy="0 0 0"/>
+                   <axis xyz="0 0 1" rpy="0 0 0"/>
                    <!-- <limit effort="100"
                           velocity="100" />
@@ -89,5 +90,5 @@
                    <child link="${prefix}talos_pan_neck_link"/>
                    <parent link="${prefix}talos_stationary_neck_link"/>
-                   <axis xyz="0 1 0" rpy="0 0 0"/>
+                   <axis xyz="0 0 1" rpy="0 0 0"/>
                    <!-- <limit effort="100"
                           velocity="100" />

Commit message: re-oriented stationary_neck_link axis to be consistent with the rest of the robot

File: robot/robot.urdf.xacro (robot description, xacro)
@@ -22,5 +22,5 @@
 	</xacro:gripper>
         <xacro:head prefix="" parent="torso_link">
-                <origin xyz="0 0 ${torso_height -neck_offset}" rpy="${PI/2} 0 0"/>
+                <origin xyz="0 0 ${torso_height - neck_offset}" rpy="0 0 0"/>
         </xacro:head>
         <!-- Add sensors to talos -->

File: urdf/head/head.urdf.xacro (robot description, xacro)
@@ -13,5 +13,5 @@
                    <xacro:inertial_template mass="${head_mass}" length="${head_mass/12}" width="${head_mass/12}" height="${head_mass/12}"/>
 		  <visual>
-			<origin xyz="0 0 0" rpy="0 -${neck_alignment} 0"/>
+			<origin xyz="0 0 0" rpy="${PI/2} 0 0"/>
 			<geometry>
                            <mesh filename="package://talos_description/meshes/head/stationary_neck.stl" scale="${scale} ${scale} ${scale}" />
@@ -79,5 +79,5 @@
                    <child link="${prefix}talos_stationary_neck_link"/>
                    <parent link="${parent}"/>
-                   <axis xyz="0 0 1" rpy="0 0 0"/>
+                   <axis xyz="0 0 1" rpy="${PI/2} 0 0"/>
                    <!-- <limit effort="100"
                           velocity="100" />
