Commit message: Added a lidar to the front of the robot

File: urdf/sensors/hokuyo.urdf.xacro (robot description, xacro)
@@ -5,5 +5,5 @@
     <joint name="${name}_joint" type="fixed">
       <axis xyz="0 1 0" />
-      <xacro:insert_block name="origin" />
+      <origin xyz="0 0 0" rpy="0 0 0"/>
       <parent link="${parent}_link"/>
       <child link="${name}_link"/>
@@ -15,4 +15,11 @@
         <inertia ixx="0.0001" ixy="0" ixz="0" iyy="0.000001" iyz="0" izz="0.0001" />
       </inertial>
+      <visual>
+         <xacro:insert_block name="origin" />
+         <geometry><mesh filename="package://talos_description/urdf/sensors/hokuyo.dae"/></geometry>
+      </visual>
+      <collision>
+         <geometry><mesh filename="package://talos_description/urdf/sensors/hokuyo.dae"/></geometry>
+      </collision>
     </link>
     <!-- gazebo extensions -->

File: urdf/sensors/sensors.urdf.xacro (robot description, xacro)
@@ -2,7 +2,9 @@
 <robot xmlns:xacro="http://ros.org/wiki/xacro">
   <xacro:include filename="$(find talos_description)/urdf/sensors/hokuyo.urdf.xacro" />
+  <xacro:property name="hokuyo_y_offset" value="-0.27"/>
+  <xacro:property name="hokuyo_z_offset" value="0.335"/>
   <xacro:macro name="talos_sensors">
       <xacro:hokuyo name="hokuyo" parent="base" ros_topic="base_scan" update_rate="50" min_angle="0" max_angle="180">
-          <origin xyz="0 1.5 1.5" rpy="0 0 0"/>
+          <origin xyz="0 ${hokuyo_y_offset} ${hokuyo_z_offset}" rpy="0 0 0"/>
       </xacro:hokuyo>
   </xacro:macro>

Commit message: Woo finally positioned lidar right

File: urdf/sensors/hokuyo.urdf.xacro (robot description, xacro)
@@ -5,5 +5,5 @@
     <joint name="${name}_joint" type="fixed">
       <axis xyz="0 1 0" />
-      <origin xyz="0 0 0" rpy="0 0 0"/>
+      <xacro:insert_block name="origin" />
       <parent link="${parent}_link"/>
       <child link="${name}_link"/>
@@ -16,8 +16,9 @@
       </inertial>
       <visual>
-         <xacro:insert_block name="origin" />
+         <origin xyz="0 0 0" rpy="0 0 0"/>
          <geometry><mesh filename="package://talos_description/urdf/sensors/hokuyo.dae"/></geometry>
       </visual>
       <collision>
+         <origin xyz="0 0 0" rpy="0 0 0"/>
          <geometry><mesh filename="package://talos_description/urdf/sensors/hokuyo.dae"/></geometry>
       </collision>

File: urdf/sensors/sensors.urdf.xacro (robot description, xacro)
@@ -2,10 +2,10 @@
 <robot xmlns:xacro="http://ros.org/wiki/xacro">
   <xacro:include filename="$(find talos_description)/urdf/sensors/hokuyo.urdf.xacro" />
-  <xacro:property name="hokuyo_y_offset" value="-0.33"/>
+  <xacro:property name="hokuyo_y_offset" value="-0.35"/>
   <xacro:property name="hokuyo_z_offset" value="0.26"/>
   <xacro:property name="hokuyo_x_offset" value="0"/>
   <xacro:macro name="talos_sensors">
-      <xacro:hokuyo name="hokuyo" parent="base" ros_topic="base_scan" update_rate="50" min_angle="0" max_angle="180">
-          <origin xyz="${hokuyo_x_offset} ${hokuyo_y_offset} ${hokuyo_z_offset}" rpy="0 0 0"/>
+      <xacro:hokuyo name="hokuyo" parent="base" ros_topic="base_scan" update_rate="50" min_angle="-1.570796" max_angle="1.570796">
+          <origin xyz="${hokuyo_x_offset} ${hokuyo_y_offset} ${hokuyo_z_offset}" rpy="0 0 -${PI/2}"/>
       </xacro:hokuyo>
   </xacro:macro>
