Commit message: Updated lidar pos

File: urdf/sensors/sensors.urdf.xacro (robot description, xacro)
@@ -2,9 +2,10 @@
 <robot xmlns:xacro="http://ros.org/wiki/xacro">
   <xacro:include filename="$(find talos_description)/urdf/sensors/hokuyo.urdf.xacro" />
-  <xacro:property name="hokuyo_y_offset" value="-0.27"/>
-  <xacro:property name="hokuyo_z_offset" value="0.335"/>
+  <xacro:property name="hokuyo_y_offset" value="-0.33"/>
+  <xacro:property name="hokuyo_z_offset" value="0.26"/>
+  <xacro:property name="hokuyo_x_offset" value="0"/>
   <xacro:macro name="talos_sensors">
       <xacro:hokuyo name="hokuyo" parent="base" ros_topic="base_scan" update_rate="50" min_angle="0" max_angle="180">
-          <origin xyz="0 ${hokuyo_y_offset} ${hokuyo_z_offset}" rpy="0 0 0"/>
+          <origin xyz="${hokuyo_x_offset} ${hokuyo_y_offset} ${hokuyo_z_offset}" rpy="0 0 0"/>
       </xacro:hokuyo>
   </xacro:macro>

Commit message: update kinect

File: urdf/sensors/sensors.urdf.xacro (robot description, xacro)
@@ -2,11 +2,18 @@
 <robot xmlns:xacro="http://ros.org/wiki/xacro">
   <xacro:include filename="$(find talos_description)/urdf/sensors/hokuyo.urdf.xacro" />
+  <xacro:include filename="$(find talos_description)/urdf/sensors/kinect.urdf.xacro" />
   <xacro:property name="hokuyo_y_offset" value="-0.35"/>
   <xacro:property name="hokuyo_z_offset" value="0.26"/>
   <xacro:property name="hokuyo_x_offset" value="0"/>
+  <xacro:property name="kinect_y_offset" value="-0.35"/>
+  <xacro:property name="kinect_z_offset" value="0.26"/>
+  <xacro:property name="kinect_x_offset" value="0"/>
   <xacro:macro name="talos_sensors">
       <xacro:hokuyo name="hokuyo" parent="base" ros_topic="base_scan" update_rate="50" min_angle="-1.570796" max_angle="1.570796">
           <origin xyz="${hokuyo_x_offset} ${hokuyo_y_offset} ${hokuyo_z_offset}" rpy="0 0 -${PI/2}"/>
       </xacro:hokuyo>
+      <xacro:kinect>
+          <origin xyz="${kinect_x_offset} ${kinect_y_offset} ${kinect_z_offset}" rpy=" 0 0 0"/>
+      </xacro:kinect>
   </xacro:macro>
 </robot>

Commit message: repositioned kinect

File: urdf/sensors/sensors.urdf.xacro (robot description, xacro)
@@ -6,7 +6,10 @@
   <xacro:property name="hokuyo_z_offset" value="0.26"/>
   <xacro:property name="hokuyo_x_offset" value="0"/>
-  <xacro:property name="kinect_y_offset" value="0"/>
-  <xacro:property name="kinect_z_offset" value="0"/>
+  <xacro:property name="kinect_y_offset" value="${0.243}"/>
+  <xacro:property name="kinect_z_offset" value="${-0.11}"/>
   <xacro:property name="kinect_x_offset" value="0"/>
+  <xacro:property name="kinect_roll_offset" value="${3*PI/2}"/>
+  <xacro:property name="kinect_pitch_offset" value="${PI/2}"/>
+  <xacro:property name="kinect_yaw_offset" value="0"/>
   <xacro:macro name="talos_sensors">
       <xacro:hokuyo name="hokuyo" parent="base" ros_topic="base_scan" update_rate="50" min_angle="-1.570796" max_angle="1.570796">
@@ -14,5 +17,5 @@
       </xacro:hokuyo>
       <xacro:kinect parent="talos_head_link">
-          <origin xyz="${kinect_x_offset} ${kinect_y_offset} ${kinect_z_offset}" rpy="0 0 0"/>
+          <origin xyz="${kinect_x_offset} ${kinect_y_offset} ${kinect_z_offset}" rpy="${kinect_roll_offset} ${kinect_pitch_offset} ${kinect_yaw_offset}"/>
       </xacro:kinect>
   </xacro:macro>
