Commit message: Added kinect still need to position it

File: urdf/sensors/kinect.gazebo.xacro (robot description, xacro)
@@ -3,5 +3,5 @@
 <xacro:macro name="kinect_camera_gazebo" params="prefix">
   <joint name="${prefix}_optical_joint" type="fixed">
-    <origin xyz="0 0 0" rpy="-1.5708 0 -1.5708"/>
+    <origin xyz="0 0 0" rpy="0 0 0"/>
     <parent link="${prefix}_link"/>
     <child link="${prefix}_frame_optical"/>
@@ -13,5 +13,5 @@
       <update_rate>20.0</update_rate>
       <camera>
-        <horizontal_fov>${60.0*M_PI/180.0}</horizontal_fov>
+        <horizontal_fov>${60.0*PI/180.0}</horizontal_fov>
         <image>
           <format>R8G8B8</format>

File: urdf/sensors/kinect.urdf.xacro (robot description, xacro)
@@ -7,5 +7,5 @@
         <inertial>
            <mass value="0.1" />
-           <origin xyz="0 0 0" rpy="0 0 0"/>
+           <xacro:insert_block name="origin"/>
            <inertia ixx="0.01"  ixy="0.0"  ixz="0.0"
                  iyy="0.01"  iyz="0.0"
@@ -26,5 +26,5 @@
     </link>
     <joint name="kinect_joint" type="fixed">
-        <origin xyz="0 0 0" rpy="0 0 0"/>
+        <origin xyz="0 0 0" rpy="${PI} 0 ${PI}"/>
         <parent link="${parent}"/>
         <child link="camera_link"/>

File: urdf/sensors/sensors.urdf.xacro (robot description, xacro)
@@ -6,6 +6,6 @@
   <xacro:property name="hokuyo_z_offset" value="0.26"/>
   <xacro:property name="hokuyo_x_offset" value="0"/>
-  <xacro:property name="kinect_y_offset" value="-0.35"/>
-  <xacro:property name="kinect_z_offset" value="0.26"/>
+  <xacro:property name="kinect_y_offset" value="0"/>
+  <xacro:property name="kinect_z_offset" value="0"/>
   <xacro:property name="kinect_x_offset" value="0"/>
   <xacro:macro name="talos_sensors">
@@ -13,6 +13,6 @@
           <origin xyz="${hokuyo_x_offset} ${hokuyo_y_offset} ${hokuyo_z_offset}" rpy="0 0 -${PI/2}"/>
       </xacro:hokuyo>
-      <xacro:kinect>
-          <origin xyz="${kinect_x_offset} ${kinect_y_offset} ${kinect_z_offset}" rpy=" 0 0 0"/>
+      <xacro:kinect parent="talos_head_link">
+          <origin xyz="${kinect_x_offset} ${kinect_y_offset} ${kinect_z_offset}" rpy="0 0 0"/>
       </xacro:kinect>
   </xacro:macro>

Commit message: Bug fix for kinect gazebo plugin

File: urdf/sensors/kinect.gazebo.xacro (robot description, xacro)
@@ -40,5 +40,5 @@
         <distortion_t1>0.0</distortion_t1>
         <distortion_t2>0.0</distortion_t2>
-        <pointCloudCutoff>0.4</pointCloudCutoff>
+        <pointCloudCutoffMax>0.4</pointCloudCutoffMax>
       </plugin>
     </sensor>

File: urdf/sensors/sensors.urdf.xacro (robot description, xacro)
@@ -6,6 +6,6 @@
   <xacro:property name="hokuyo_z_offset" value="0.26"/>
   <xacro:property name="hokuyo_x_offset" value="0"/>
-  <xacro:property name="kinect_y_offset" value="0"/>
-  <xacro:property name="kinect_z_offset" value="0"/>
+  <xacro:property name="kinect_y_offset" value="0.24"/>
+  <xacro:property name="kinect_z_offset" value="-0.125"/>
   <xacro:property name="kinect_x_offset" value="0"/>
   <xacro:macro name="talos_sensors">
@@ -14,5 +14,5 @@
       </xacro:hokuyo>
       <xacro:kinect parent="talos_tilt_head_link">
-          <origin xyz="${kinect_x_offset} ${kinect_y_offset} ${kinect_z_offset}" rpy="0 0 0"/>
+          <origin xyz="${kinect_x_offset} ${kinect_y_offset} ${kinect_z_offset}" rpy="0 ${PI/2} ${PI/2}"/>
       </xacro:kinect>
   </xacro:macro>
