Commit message: re-oriented kinect to be inside the head again

File: urdf/sensors/kinect.urdf.xacro (robot description, xacro)
@@ -2,4 +2,6 @@
 <robot xmlns:xacro="http://ros.org/wiki/xacro">
   <xacro:include filename="$(find talos_description)/urdf/sensors/kinect.gazebo.xacro" />
+  <xacro:property name="kinect_z_offset" value="0.005"/>
+  <xacro:property name="kinect_y_offset" value="0.06"/>
   <xacro:macro name="kinect" params="*origin parent">
     <!-- still need kinect models and links -->
@@ -26,5 +28,5 @@
     </link>
     <joint name="kinect_joint" type="fixed">
-        <origin xyz="0 0 0" rpy="${PI} 0 ${PI}"/>
+        <origin xyz="0 ${kinect_y_offset} ${kinect_z_offset}" rpy="0 0 0"/>
         <parent link="${parent}"/>
         <child link="camera_link"/>

File: urdf/sensors/sensors.urdf.xacro (robot description, xacro)
@@ -6,7 +6,7 @@
   <xacro:property name="hokuyo_z_offset" value="0.26"/>
   <xacro:property name="hokuyo_x_offset" value="0"/>
-  <xacro:property name="kinect_y_offset" value="0.24"/>
+  <!--<xacro:property name="kinect_y_offset" value="0.24"/>
   <xacro:property name="kinect_z_offset" value="-0.125"/>
-  <xacro:property name="kinect_x_offset" value="0"/>
+  <xacro:property name="kinect_x_offset" value="0"/>-->
   <xacro:macro name="talos_sensors">
       <xacro:hokuyo name="hokuyo" parent="base" ros_topic="base_scan" update_rate="50" min_angle="-1.570796" max_angle="1.570796">
@@ -14,5 +14,5 @@
       </xacro:hokuyo>
       <xacro:kinect parent="talos_tilt_head_link">
-          <origin xyz="${kinect_x_offset} ${kinect_y_offset} ${kinect_z_offset}" rpy="0 ${PI/2} ${PI/2}"/>
+          <origin xyz="0 0 0" rpy="0 0 ${PI/2}"/>
       </xacro:kinect>
   </xacro:macro>
