Commit message: Updated physics values

File: urdf/base/base.urdf.xacro (robot description, xacro)
@@ -3,5 +3,5 @@
 	<xacro:property name="base_width" value="0.62265" />
 	<xacro:property name="base_height" value="0.37817" />
-	<xacro:property name="base_mass" value="0.22" />
+	<xacro:property name="base_mass" value="8.20" />
 	<xacro:macro name="base" params="name">
 		<link name="${name}_link">

File: urdf/torso/torso.urdf.xacro (robot description, xacro)
@@ -3,5 +3,5 @@
 	<xacro:property name="torso_width" value="0.4324" />
 	<xacro:property name="torso_height" value="1.00318" />
-	<xacro:property name="torso_mass" value="0.22" />
+	<xacro:property name="torso_mass" value="5.20" />
 	<xacro:macro name="torso" params="name parent *origin">
 		<link name="${name}_link">

Commit message: Stable wheel bases now

File: urdf/base/base.urdf.xacro (robot description, xacro)
@@ -24,14 +24,14 @@
 		</link>
                 <xacro:wheel prefix="fl" parent="base_link">
-                    <origin xyz="${base_width/3} ${base_width/3} 0" rpy="0 ${PI/2} 0"/>
+                    <origin xyz="${base_width/3} ${base_width/3} 0" rpy="0 ${PI/2} ${PI/2}"/>
                 </xacro:wheel>
                 <xacro:wheel prefix="fr" parent="base_link">
-                    <origin xyz="${-base_width/3} ${base_width/3} 0" rpy="0 ${PI/2} 0"/>
+                    <origin xyz="${-base_width/3} ${base_width/3} 0" rpy="0 ${PI/2} ${PI/2}"/>
                 </xacro:wheel>
                 <xacro:wheel prefix="bl" parent="base_link">
-                    <origin xyz="${base_width/3} ${-base_width/3} 0" rpy="0 ${PI/2} 0"/>
+                    <origin xyz="${base_width/3} ${-base_width/3} 0" rpy="0 ${PI/2} ${PI/2}"/>
                 </xacro:wheel>
                 <xacro:wheel prefix="br" parent="base_link">
-                   <origin xyz="${-base_width/3} ${-base_width/3} 0" rpy="0 ${PI/2} 0"/>
+                   <origin xyz="${-base_width/3} ${-base_width/3} 0" rpy="0 ${PI/2} ${PI/2}"/>
                 </xacro:wheel>
 		<xacro:talos_wheel_transmission prefix="bl"/>

File: urdf/wheel/wheel.urdf.xacro (robot description, xacro)
@@ -11,5 +11,5 @@
 			<origin xyz="0 0 0" rpy="0 0 0"/>
 			<geometry>
-			  <cylinder length="${wheel_height}" radius="${wheel_radius}" />
+			  <cylinder length="${wheel_height*1.5}" radius="${wheel_radius}" />
 			</geometry>
 			<material name="white"/>
@@ -18,5 +18,5 @@
 			<origin xyz="0 0 0" rpy="0 0 0"/>
 			<geometry>
-			  <cylinder length="${wheel_height}" radius="${wheel_radius}" />
+			  <cylinder length="${wheel_height*1.5}" radius="${wheel_radius}" />
 			</geometry>
 		  </collision>

Commit message: added wheel visuals and joints

File: urdf/base/base.urdf.xacro (robot description, xacro)
@@ -1,5 +1,6 @@
 <?xml version="1.0"?>
 <robot xmlns:xacro="http://www.ros.org/wiki/xacro">
-        <xacro:include filename="$(find talos_description)/urdf/wheel/wheel.urdf.xacro" />
+        <xacro:include filename="$(find talos_description)/urdf/wheel/back_wheel.urdf.xacro" />
+	<xacro:include filename="$(find talos_description)/urdf/wheel/caster_wheel.urdf.xacro" />
         <xacro:include filename="$(find talos_description)/urdf/wheel/wheel.transmission.xacro" />
 	<xacro:property name="base_width" value="0.62265" />
@@ -7,4 +8,9 @@
 	<xacro:property name="base_skirt_height_guestimate" value="0.073" />
 	<xacro:property name="base_mass" value="8.20" />
+	<xacro:property name="caster_to_side_offset" value="0.2175" />
+	<xacro:property name="caster_to_front_offset" value="0.21745" />
+	<xacro:property name="back_wheel_to_side_offset" value="0.229125" />
+	<xacro:property name="back_wheel_to_back_offset" value="0.2" />
+	<xacro:property name="back_wheel_vertical_offset" value="0.040132" />
 	<xacro:macro name="base" params="name">
 		<link name="${name}_link">
@@ -24,16 +30,16 @@
 		  <xacro:inertial_template mass="${base_mass}" length="${base_width}" width="${base_width}" height="${base_height}"/>
 		</link>
-                <xacro:wheel prefix="fl" parent="base_link">
-                    <origin xyz="${base_width/3} ${base_width/3} 0" rpy="0 ${PI/2} ${PI/2}"/>
-                </xacro:wheel>
-                <xacro:wheel prefix="fr" parent="base_link">
-                    <origin xyz="${-base_width/3} ${base_width/3} 0" rpy="0 ${PI/2} ${PI/2}"/>
-                </xacro:wheel>
-                <xacro:wheel prefix="bl" parent="base_link">
-                    <origin xyz="${base_width/3} ${-base_width/3} 0" rpy="0 ${PI/2} ${PI/2}"/>
-                </xacro:wheel>
-                <xacro:wheel prefix="br" parent="base_link">
-                   <origin xyz="${-base_width/3} ${-base_width/3} 0" rpy="0 ${PI/2} ${PI/2}"/>
-                </xacro:wheel>
+                <xacro:caster_wheel prefix="fl" parent="base_link">
+                    <origin xyz="${caster_to_side_offset} ${caster_to_front_offset} 0" rpy="0 0 0"/>
+                </xacro:caster_wheel>
+                <xacro:caster_wheel prefix="fr" parent="base_link">
+                    <origin xyz="${-caster_to_side_offset} ${caster_to_front_offset} 0" rpy="0 0 0"/>
+                </xacro:caster_wheel>
+                <xacro:back_wheel prefix="bl" parent="base_link">
+                    <origin xyz="${back_wheel_to_side_offset} ${-back_wheel_to_back_offset} -${back_wheel_vertical_offset}" rpy="0 0 0"/>
+                </xacro:back_wheel>
+                <xacro:back_wheel prefix="br" parent="base_link">
+                   <origin xyz="${-back_wheel_to_side_offset} ${-back_wheel_to_back_offset} -${back_wheel_vertical_offset}" rpy="0 0 0"/>
+                </xacro:back_wheel>
 		<xacro:talos_wheel_transmission prefix="bl"/>
 		<xacro:talos_wheel_transmission prefix="br"/>

Commit message: fixed collision elements for torso, caster, and gripper

File: urdf/base/base.urdf.xacro (robot description, xacro)
@@ -23,5 +23,5 @@
 		  </visual>
 		  <collision>
-			<origin xyz="0 0 ${base_height/2}" rpy="0 0 0"/>
+			<origin xyz="0 0 ${base_height/2 - base_skirt_height_guestimate}" rpy="0 0 0"/>
 			<geometry>
 			  <box size="${base_width} ${base_width} ${base_height}" />

File: urdf/gripper/gripper.urdf.xacro (robot description, xacro)
@@ -4,4 +4,5 @@
 	<xacro:property name="gripper_base_length" value="0.08316" />
 	<xacro:property name="gripper_base_width" value="0.0889" />
+	<xacro:property name="gripper_base_radius" value="0.04445" />
 	<xacro:property name="gripper_base_height" value="0.0889" />
 	<xacro:property name="gripper_base_mass" value="0.22" />
@@ -26,7 +27,7 @@
 		 </visual>
 		 <collision>
-		  <origin xyz="0 ${gripper_base_length/2} -${gripper_base_height/2}" rpy="0 0 0"/>
+		  <origin xyz="0 ${gripper_base_length/2} 0" rpy="${PI/2} 0 0"/>
 		  <geometry>
-		   <box size="${gripper_base_width} ${gripper_base_length} ${gripper_base_height}" />
+		   <cylinder length="${gripper_base_length}" radius="${gripper_base_radius}" />
 		  </geometry>
 		 </collision>
@@ -42,7 +43,7 @@
 		 </visual>
 		 <collision>
-		  <origin xyz="0 ${stationary_claw_length/2} 0" rpy="0 0 0"/>
+		  <origin xyz="${stationary_claw_width/2} 0 -${1.25*gripper_base_width/2}" rpy="0 -${PI/2} 0"/>
 		  <geometry>
-		   <box size="${stationary_claw_width} ${stationary_claw_length} ${stationary_claw_height}" /> <!-- will probably need a better collision element-->
+		   <mesh filename="package://talos_description/meshes/gripper/stationary_claw_link.stl" scale="${scale} ${scale} ${scale}"/>
 		  </geometry>
 		 </collision>
@@ -58,7 +59,7 @@
 		 </visual>
 		 <collision>
-		  <origin xyz="0 ${wrist_length/2 - wrist_offset} 0" rpy="0 0 0"/>
+		  <origin xyz="${movable_claw_width/2 + 0.002} -0.01 0.025" rpy="0 ${PI} 0"/>
 		  <geometry>
-		   <box size="${wrist_width} ${wrist_length} ${wrist_height}" />
+			 <mesh filename="package://talos_description/meshes/gripper/movable_claw_link.stl" scale="${scale} ${scale} ${scale}"/>
 		  </geometry>
 		 </collision>

File: urdf/wheel/caster_wheel.urdf.xacro (robot description, xacro)
@@ -43,5 +43,5 @@
 		  </visual>
 		  <collision>
-                        <origin xyz="0 0 ${caster_height/2 - caster_vertical_offset}" rpy="0 0 0"/>
+                        <origin xyz="0 ${-caster_horizontal_offset_inc_guess} ${caster_height/2 - caster_vertical_offset - caster_vertical_offset_inc_guess}" rpy="0 0 0"/>
 			<geometry>
 			  <box size="${caster_width} ${caster_length} ${caster_height}" />

Commit message: First commit of updating hwiface

File: urdf/base/base.urdf.xacro (robot description, xacro)
@@ -3,5 +3,6 @@
         <xacro:include filename="$(find talos_description)/urdf/wheel/back_wheel.urdf.xacro" />
 	<xacro:include filename="$(find talos_description)/urdf/wheel/caster_wheel.urdf.xacro" />
-        <xacro:include filename="$(find talos_description)/urdf/wheel/wheel.transmission.xacro" />
+        <xacro:include filename="$(find talos_description)/urdf/wheel/back_wheel.transmission.xacro" />
+        <xacro:include filename="$(find talos_description)/urdf/wheel/caster_wheel.transmission.xacro" />
 	<xacro:property name="base_width" value="0.62265" />
 	<xacro:property name="base_height" value="0.37817" />
@@ -42,8 +43,8 @@
                    <origin xyz="${-back_wheel_to_side_offset} ${-back_wheel_to_back_offset} -${back_wheel_vertical_offset}" rpy="0 0 0"/>
                 </xacro:back_wheel>
-		<xacro:talos_wheel_transmission prefix="bl"/>
-		<xacro:talos_wheel_transmission prefix="br"/>
-		<xacro:talos_wheel_transmission prefix="fr"/>
-                <xacro:talos_wheel_transmission prefix="fl"/>
+		<xacro:caster_wheel_transmission prefix="fl"/>
+		<xacro:caster_wheel_transmission prefix="fr"/>
+		<xacro:back_wheel_transmission prefix="br"/>
+                <xacro:back_wheel_transmission prefix="bl"/>
 	</xacro:macro>
 </robot>

File: urdf/torso/torso.urdf.xacro (robot description, xacro)
@@ -4,5 +4,5 @@
 	<xacro:property name="torso_height" value="1.03818" />
 	<xacro:property name="torso_mass" value="5.20" />
-	<xacro:property name="torso_offset" value="0.23965" />
+	<xacro:property name="torso_offset" value="0.33965" />
         <xacro:include filename="$(find talos_description)/urdf/torso/torso.transmission.xacro"/>
 	<xacro:macro name="torso" params="name parent *origin">
@@ -11,5 +11,4 @@
 		  <origin xyz="-${torso_width/2} ${torso_width/2} -${torso_offset}" rpy="0 0 -${PI/2}"/>
 		  <geometry>
-			 <!--<box size="${torso_width} ${torso_width} ${torso_height}" />-->
 <mesh filename="package://talos_description/meshes/torso/torso_link.stl" scale="${scale} ${scale} ${scale}"/>
 		  </geometry>
@@ -29,5 +28,5 @@
 		 <parent link="${parent}_link" />
 		 <child link="${name}_link" />
-		 <insert_block name="origin"/>
+		 <xacro:insert_block name="origin"/>
 		 <!--<origin xyz="0 0 ${base_height}" rpy="0 0 0"/>-->
 		</joint>

Commit message: slightly shifted positions of base, caster, caster wheels

File: urdf/base/base.urdf.xacro (robot description, xacro)
@@ -16,5 +16,4 @@
 		<link name="${name}_link">
 		  <visual>
-			<origin xyz="${base_width/2} ${base_width/2} 0" rpy="0 0 ${PI}"/>
 			<geometry>
 			  <mesh filename="package://talos_description/meshes/base/base_link.stl" scale="${scale} ${scale} ${scale}"/>

File: urdf/wheel/back_wheel.urdf.xacro (robot description, xacro)
@@ -9,5 +9,5 @@
                    <xacro:inertial_template mass="${back_wheel_mass}" length="${back_wheel_width}" width="${back_wheel_radius}" height="${back_wheel_width}"/>
 		  <visual>
-			<origin xyz="${-back_wheel_width/2} ${-back_wheel_radius} ${-back_wheel_radius}" rpy="0 0 0"/>
+			<origin xyz="${-back_wheel_width/2 - 0.003} ${-back_wheel_radius} ${-back_wheel_radius}" rpy="0 0 0"/>
 			<geometry>
                           <!--<cylinder length="${back_wheel_width}" radius="${back_wheel_radius}" />-->

File: urdf/wheel/caster_wheel.urdf.xacro (robot description, xacro)
@@ -3,5 +3,5 @@
 	<!--need to update caster and caster wheel masses-->
 	<xacro:property name="caster_wheel_radius" value="0.04435" />
-	<xacro:property name="caster_wheel_width" value="0.0381" />
+	<xacro:property name="caster_wheel_width" value="0.02755" />
 	<xacro:property name="caster_wheel_mass" value="1.20" />
 	<xacro:property name="caster_width" value="0.06274" />
@@ -35,5 +35,5 @@
                    <xacro:inertial_template mass="${caster_mass}" length="${caster_length}" width="${caster_width}" height="${caster_height}"/>
 		  <visual>
-			<origin xyz="${-caster_width/2} ${-caster_horizontal_offset+caster_horizontal_offset_inc_guess} ${-caster_vertical_offset-caster_vertical_offset_inc_guess} " rpy="0 0 ${-PI/2}"/>
+			<origin xyz="0 0 0" rpy="0 0 0"/>
 			<geometry>
                           <mesh filename="package://talos_description/meshes/wheel/caster.stl" scale="${scale} ${scale} ${scale}" />
@@ -42,8 +42,13 @@
 		  </visual>
 		  <collision>
-                        <origin xyz="0 ${-caster_horizontal_offset_inc_guess} ${caster_height/2 - caster_vertical_offset - caster_vertical_offset_inc_guess}" rpy="0 0 0"/>
+			<origin xyz="0 0 0" rpy="0 0 0"/>
+			<geometry>
+                          <mesh filename="package://talos_description/meshes/wheel/caster.stl" scale="${scale} ${scale} ${scale}" />
+			</geometry>
+			<material name="white"/>
+                        <!--<origin xyz="0 ${-caster_horizontal_offset_inc_guess} ${caster_height/2 - caster_vertical_offset - caster_vertical_offset_inc_guess}" rpy="0 0 0"/>
 			<geometry>
 			  <box size="${caster_width} ${caster_length} ${caster_height}" />
-			</geometry>
+			</geometry>-->
 		  </collision>
 		</link>

Commit message: Added physics vals

File: urdf/base/base.urdf.xacro (robot description, xacro)
@@ -8,5 +8,5 @@
 	<xacro:property name="base_height" value="0.37817" />
 	<xacro:property name="base_skirt_height_guestimate" value="0.073" />
-	<xacro:property name="base_mass" value="8.20" />
+	<xacro:property name="base_mass" value="15.00" />
 	<xacro:property name="caster_to_side_offset" value="0.2175" />
 	<xacro:property name="caster_to_front_offset" value="0.21745" />
@@ -42,6 +42,6 @@
                    <origin xyz="${-back_wheel_to_side_offset} ${-back_wheel_to_back_offset} -${back_wheel_vertical_offset}" rpy="0 0 0"/>
                 </xacro:back_wheel>
-		<xacro:caster_wheel_transmission prefix="fl"/>
-		<xacro:caster_wheel_transmission prefix="fr"/>
+		<!-- <xacro:caster_wheel_transmission prefix="fl"/> -->
+		<!-- <xacro:caster_wheel_transmission prefix="fr"/> -->
 		<xacro:back_wheel_transmission prefix="br"/>
                 <xacro:back_wheel_transmission prefix="bl"/>

File: urdf/wheel/caster_wheel.urdf.xacro (robot description, xacro)
@@ -16,5 +16,5 @@
 		<link name="${prefix}_caster_wheel_link">
                   <mass value="${caster_wheel_mass}"/>
-                   <xacro:inertial_template mass="${caster_wheel_mass}" length="${caster_wheel_width}" width="${caster_wheel_radius}" height="${caster_wheel_width}"/>
+                   <xacro:inertial_template mass="${caster_wheel_mass*10}" length="${caster_wheel_width*10}" width="${caster_wheel_radius*10}" height="${caster_wheel_width*10}"/>
 		  <visual>
 			<origin xyz="0 0 0" rpy="0 0 0"/>
@@ -69,6 +69,6 @@
                 <gazebo reference="${prefix}_caster_wheel_link">
                      <!-- <selfCollide>true</selfCollide> -->
-		     <mu1 value="0.0"/>
-	             <mu2 value="0.0"/>
+		     <mu1 value="0.3"/>
+	             <mu2 value="0.3"/>
 		     <!-- <kp value="100000.0" />
 	             <kd value="1.0" /> -->

Commit message: Revert "Adding details"

File: urdf/base/base.urdf.xacro (robot description, xacro)
@@ -17,4 +17,5 @@
 		<link name="${name}_link">
 		  <visual>
+			<origin xyz="${base_width/2} ${base_width/2} 0" rpy="0 0 ${PI}"/>
 			<geometry>
 			  <mesh filename="package://talos_description/meshes/base/base_link.stl" scale="${scale} ${scale} ${scale}"/>

File: urdf/wheel/back_wheel.urdf.xacro (robot description, xacro)
@@ -1,16 +1,16 @@
 <?xml version="1.0"?>
 <robot xmlns:xacro="http://www.ros.org/wiki/xacro">
-	<xacro:property name="back_wheel_radius" value="0.0762" />
-	<xacro:property name="back_wheel_width" value="0.0127" />
+	<xacro:property name="back_wheel_radius" value="0.072805" />
+	<xacro:property name="back_wheel_height" value="0.0381" />
 	<xacro:property name="back_wheel_mass" value="1.20" />
 	<xacro:macro name="back_wheel" params="prefix *origin parent">
 		<link name="${prefix}_back_wheel_link">
                   <mass value="${back_wheel_mass}"/>
-                   <xacro:inertial_template mass="${back_wheel_mass}" length="${back_wheel_width}" width="${back_wheel_radius}" height="${back_wheel_width}"/>
+                   <xacro:inertial_template mass="${back_wheel_mass}" length="${back_wheel_height}" width="${back_wheel_radius}" height="${back_wheel_height}"/>
 		  <visual>
-			<origin xyz="${-back_wheel_width/2 - 0.003} ${-back_wheel_radius} ${-back_wheel_radius}" rpy="0 0 0"/>
+			<origin xyz="0 0 0" rpy="0 ${PI/2} 0"/>
 			<geometry>
-                          <!--<cylinder length="${back_wheel_width}" radius="${back_wheel_radius}" />-->
-			  <mesh filename="package://talos_description/meshes/wheel/back_wheel.stl" scale="${scale} ${scale} ${scale}" />
+                          <cylinder length="${back_wheel_height}" radius="${back_wheel_radius}" />
+			  <!-- <mesh filename="package://talos_description/meshes/wheel/back_wheel.stl" scale="${scale} ${scale} ${scale}" /> -->
 			</geometry>
 			<material name="white"/>
@@ -19,5 +19,5 @@
                         <origin xyz="0 0 0" rpy="0 ${PI/2} 0"/>
 			<geometry>
-			  <cylinder length="${back_wheel_width}" radius="${back_wheel_radius}" />
+			  <cylinder length="${back_wheel_height}" radius="${back_wheel_radius}" />
 			</geometry>
 		  </collision>

File: urdf/wheel/caster_wheel.urdf.xacro (robot description, xacro)
@@ -2,6 +2,6 @@
 <robot xmlns:xacro="http://www.ros.org/wiki/xacro">
 	<!--need to update caster and caster wheel masses-->
-	<xacro:property name="caster_wheel_radius" value="0.04435" />
-	<xacro:property name="caster_wheel_width" value="0.02755" />
+	<xacro:property name="caster_wheel_radius" value="0.0415" />
+	<xacro:property name="caster_wheel_width" value="0.02675" />
 	<xacro:property name="caster_wheel_mass" value="1.20" />
 	<xacro:property name="caster_width" value="0.06274" />
@@ -18,7 +18,8 @@
                    <xacro:inertial_template mass="${caster_wheel_mass*10}" length="${caster_wheel_width*10}" width="${caster_wheel_radius*10}" height="${caster_wheel_width*10}"/>
 		  <visual>
-			<origin xyz="0 0 0" rpy="0 0 0"/>
+			<origin xyz="0 0 0" rpy="0 ${-PI/2} 0"/>
 			<geometry>
-			  <mesh filename="package://talos_description/meshes/wheel/caster_wheel.stl" scale="${scale} ${scale} ${scale}" />
+			  <cylinder length="${caster_wheel_width}" radius="${caster_wheel_radius}" />
+			  <!--<mesh filename="package://talos_description/meshes/wheel/caster_wheel.stl" scale="${scale} ${scale} ${scale}" />-->
 			</geometry>
 			<material name="white"/>
@@ -35,5 +36,5 @@
                    <xacro:inertial_template mass="${caster_mass}" length="${caster_length}" width="${caster_width}" height="${caster_height}"/>
 		  <visual>
-			<origin xyz="0 0 0" rpy="0 0 0"/>
+			<origin xyz="${-caster_width/2} ${-caster_horizontal_offset+caster_horizontal_offset_inc_guess} ${-caster_vertical_offset-caster_vertical_offset_inc_guess} " rpy="0 0 ${-PI/2}"/>
 			<geometry>
                           <mesh filename="package://talos_description/meshes/wheel/caster.stl" scale="${scale} ${scale} ${scale}" />
@@ -42,13 +43,8 @@
 		  </visual>
 		  <collision>
-			<origin xyz="0 0 0" rpy="0 0 0"/>
-			<geometry>
-                          <mesh filename="package://talos_description/meshes/wheel/caster.stl" scale="${scale} ${scale} ${scale}" />
-			</geometry>
-			<material name="white"/>
-                        <!--<origin xyz="0 ${-caster_horizontal_offset_inc_guess} ${caster_height/2 - caster_vertical_offset - caster_vertical_offset_inc_guess}" rpy="0 0 0"/>
+                        <origin xyz="0 ${-caster_horizontal_offset_inc_guess} ${caster_height/2 - caster_vertical_offset - caster_vertical_offset_inc_guess}" rpy="0 0 0"/>
 			<geometry>
 			  <box size="${caster_width} ${caster_length} ${caster_height}" />
-			</geometry>-->
+			</geometry>
 		  </collision>
 		</link>
