Commit message: Added head transmission

File: urdf/head/head.transmission.xacro (robot description, xacro)
@@ -1,5 +1,5 @@
 <?xml version="1.0"?>
 <robot xmlns:xacro="http://www.ros.org/wiki/xacro">
-  <xacro:macro name="talos_gripper_transmission" params="prefix">
+  <xacro:macro name="talos_head_transmission" params="prefix">
     <transmission name="${prefix}talos_head_joint_trans">
     <type>transmission_interface/SimpleTransmission</type>

File: urdf/head/head.urdf.xacro (robot description, xacro)
@@ -68,4 +68,5 @@
 	       </gazebo>
          <xacro:include filename="$(find talos_description)/urdf/head/head.transmission.xacro" />
+         <xacro:talos_head_transmission prefix=""/>
 	</xacro:macro>
 </robot>

Commit message: updated model

File: urdf/head/head.transmission.xacro (robot description, xacro)
@@ -5,9 +5,9 @@
     <type>transmission_interface/SimpleTransmission</type>
     <joint name="${prefix}talos_head_joint">
-       <hardwareInterface>EffortJointInterface</hardwareInterface>
+       <hardwareInterface>PositionJointInterface</hardwareInterface>
     </joint>
     <actuator name="${prefix}talos_head_joint_motor">
       <mechanicalReduction>1</mechanicalReduction>
-      <hardwareInterface>EffortJointInterface</hardwareInterface>
+      <hardwareInterface>PositionJointInterface</hardwareInterface>
     </actuator>
   </transmission>
@@ -15,9 +15,9 @@
       <type>transmission_interface/SimpleTransmission</type>
       <joint name="${prefix}talos_neck_joint">
-        <hardwareInterface>EffortJointInterface</hardwareInterface>
+        <hardwareInterface>PositionJointInterface</hardwareInterface>
       </joint>
       <actuator name="${prefix}talos_neck_joint_motor">
         <mechanicalReduction>1</mechanicalReduction>
-        <hardwareInterface>EffortJointInterface</hardwareInterface>
+        <hardwareInterface>PositionJointInterface</hardwareInterface>
       </actuator>
     </transmission>

File: urdf/head/head.urdf.xacro (robot description, xacro)
@@ -1,5 +1,6 @@
 <?xml version="1.0"?>
 <robot xmlns:xacro="http://www.ros.org/wiki/xacro">
-	<xacro:property name="head_mass" value="1.20" />
+	<xacro:property name="head_mass" value="0.20" />
+         <xacro:include filename="$(find talos_description)/urdf/head/head.transmission.xacro" />
 	<xacro:macro name="head" params="prefix parent *origin">
                 <!-- head which attackes to the pan unit, this is the tilt unit -->
@@ -67,5 +68,4 @@
                      <selfCollide>true</selfCollide>
 	       </gazebo>
-         <xacro:include filename="$(find talos_description)/urdf/head/head.transmission.xacro" />
          <xacro:talos_head_transmission prefix=""/>
 	</xacro:macro>

File: urdf/wheel/caster_wheel.transmission.xacro (robot description, xacro)
@@ -6,9 +6,9 @@
 	    <type>transmission_interface/SimpleTransmission</type>
 	    <joint name="${prefix}_caster_to_wheel">
-               <hardwareInterface>VelocityJointInterface</hardwareInterface>
+               <hardwareInterface>JointStateInterface</hardwareInterface>
             </joint>
 	    <actuator name="${prefix}_caster_to_wheel_motor">
 	      <mechanicalReduction>1</mechanicalReduction>
-              <hardwareInterface>VelocityJointInterface</hardwareInterface>
+              <hardwareInterface>JointStateInterface</hardwareInterface>
 	    </actuator>
 	  </transmission>
@@ -16,9 +16,9 @@
 	    <type>transmission_interface/SimpleTransmission</type>
 	    <joint name="${prefix}_base_link_to_caster">
-               <hardwareInterface>VelocityJointInterface</hardwareInterface>
+               <hardwareInterface>JointStateInterface</hardwareInterface>
             </joint>
 	    <actuator name="${prefix}_base_link_to_caster_motor">
 	      <mechanicalReduction>1</mechanicalReduction>
-              <hardwareInterface>VelocityJointInterface</hardwareInterface>
+              <hardwareInterface>JointStateInterface</hardwareInterface>
 	    </actuator>
 	  </transmission>

Commit message: Added transmissions for head

File: urdf/head/head.transmission.xacro (robot description, xacro)
@@ -2,20 +2,20 @@
 <robot xmlns:xacro="http://www.ros.org/wiki/xacro">
   <xacro:macro name="talos_head_transmission" params="prefix">
-    <transmission name="${prefix}talos_head_joint_trans">
+    <transmission name="${prefix}talos_pan_neck_joint_trans">
     <type>transmission_interface/SimpleTransmission</type>
-    <joint name="${prefix}talos_head_joint">
+    <joint name="${prefix}talos_pan_neck_joint">
        <hardwareInterface>PositionJointInterface</hardwareInterface>
     </joint>
-    <actuator name="${prefix}talos_head_joint_motor">
+    <actuator name="${prefix}talos_pan_neck_joint_motor">
       <mechanicalReduction>1</mechanicalReduction>
       <hardwareInterface>PositionJointInterface</hardwareInterface>
     </actuator>
   </transmission>
-    <transmission name="${prefix}talos_neck_joint_trans">
+   <transmission name="${prefix}talos_tilt_head_joint_trans">
       <type>transmission_interface/SimpleTransmission</type>
-      <joint name="${prefix}talos_neck_joint">
+      <joint name="${prefix}talos_tilt_head_joint">
         <hardwareInterface>PositionJointInterface</hardwareInterface>
       </joint>
-      <actuator name="${prefix}talos_neck_joint_motor">
+      <actuator name="${prefix}talos_tilt_head_joint_motor">
         <mechanicalReduction>1</mechanicalReduction>
         <hardwareInterface>PositionJointInterface</hardwareInterface>

File: urdf/head/head.urdf.xacro (robot description, xacro)
@@ -96,5 +96,5 @@
                                      friction="0.0" /> -->
                </joint>
-               <gazebo reference="${prefix}talos_pan_neck_link">
+               <!-- <gazebo reference="${prefix}talos_pan_neck_link">
                      <selfCollide>true</selfCollide>
 	       </gazebo>
@@ -104,5 +104,5 @@
                <gazebo reference="${prefix}talos_stationary_neck_link">
                      <selfCollide>true</selfCollide>
-	       </gazebo>
+	       </gazebo> TODO: put inside .gazebo file -->
          <xacro:talos_head_transmission prefix=""/>
 	</xacro:macro>
