Commit message: Updating pid, masses, and inertias

File: urdf/head/head.urdf.xacro (robot description, xacro)
@@ -1,5 +1,5 @@
 <?xml version="1.0"?>
 <robot xmlns:xacro="http://www.ros.org/wiki/xacro">
-	<xacro:property name="head_mass" value="0.20" />
+	<xacro:property name="head_mass" value="1.20" />
         <xacro:property name="neck_offset" value="0.085" />
         <xacro:property name="head_offset" value="0.075" />
@@ -10,5 +10,5 @@
 		<link name="${prefix}talos_head_link">
                   <mass value="${head_mass}"/>
-                   <xacro:inertial_template mass="${head_mass}" length="${head_mass}" width="${head_mass}" height="${head_mass}"/>
+                   <xacro:inertial_template mass="${head_mass/12}" length="${head_mass/12}" width="${head_mass/12}" height="${head_mass/12}"/>
 		  <visual>
 			<origin xyz="0 ${head_offset} 0" rpy="0 0 0"/>
@@ -28,5 +28,5 @@
               <link name="${prefix}talos_neck_link">
                   <mass value="${head_mass}"/>
-                   <xacro:inertial_template mass="${head_mass}" length="${head_mass}" width="${head_mass}" height="${head_mass}"/>
+                   <xacro:inertial_template mass="${head_mass/12}" length="${head_mass/12}" width="${head_mass/12}" height="${head_mass/12}"/>
 		  <visual>
 			<origin xyz="0 0 0" rpy="0 -${neck_alignment} 0"/>

Commit message: Disabled head joints due to improper modelling on my part

File: urdf/head/head.urdf.xacro (robot description, xacro)
@@ -1,5 +1,5 @@
 <?xml version="1.0"?>
 <robot xmlns:xacro="http://www.ros.org/wiki/xacro">
-	<xacro:property name="head_mass" value="1.20" />
+	<xacro:property name="head_mass" value="0.20" />
         <xacro:property name="neck_offset" value="0.085" />
         <xacro:property name="head_offset" value="0.075" />
@@ -10,5 +10,5 @@
 		<link name="${prefix}talos_head_link">
                   <mass value="${head_mass}"/>
-                   <xacro:inertial_template mass="${head_mass/12}" length="${head_mass/12}" width="${head_mass/12}" height="${head_mass/12}"/>
+                   <xacro:inertial_template mass="${head_mass}" length="${head_mass/12}" width="${head_mass/12}" height="${head_mass/12}"/>
 		  <visual>
 			<origin xyz="0 ${head_offset} 0" rpy="0 0 0"/>
@@ -28,5 +28,5 @@
               <link name="${prefix}talos_neck_link">
                   <mass value="${head_mass}"/>
-                   <xacro:inertial_template mass="${head_mass/12}" length="${head_mass/12}" width="${head_mass/12}" height="${head_mass/12}"/>
+                   <xacro:inertial_template mass="${head_mass}" length="${head_mass/12}" width="${head_mass/12}" height="${head_mass/12}"/>
 		  <visual>
 			<origin xyz="0 0 0" rpy="0 -${neck_alignment} 0"/>
@@ -44,24 +44,24 @@
 		</link>
                <!-- Join head to neck (Tilt unit) -->
-               <joint name="${prefix}talos_head_joint" type="revolute">
+               <joint name="${prefix}talos_head_joint" type="fixed">
                    <origin xyz="0 0 0" rpy="0 0 0"/>
                    <child link="${prefix}talos_head_link"/>
                    <parent link="${prefix}talos_neck_link"/>
                    <axis xyz="0 1 0" rpy="0 0 0"/>
-                   <limit effort="100"
+                   <!-- <limit effort="100"
                           velocity="100" />
                    <joint_properties damping="0.0"
-                                     friction="0.0" />
+                                     friction="0.0" /> -->
                </joint>
                <!-- Join neck to torso (Pan unit) -->
-               <joint name="${prefix}talos_neck_joint" type="continuous">
+               <joint name="${prefix}talos_neck_joint" type="fixed">
                    <xacro:insert_block name="origin"/>
                    <child link="${prefix}talos_neck_link"/>
                    <parent link="${parent}"/>
                    <axis xyz="0 1 0" rpy="0 0 0"/>
-                   <limit effort="100"
+                   <!-- <limit effort="100"
                           velocity="100" />
                    <joint_properties damping="0.0"
-                                     friction="0.0" />
+                                     friction="0.0" /> -->
                </joint>
                <gazebo reference="${prefix}talos_head_link">

Commit message: Head revamp

File: urdf/head/head.urdf.xacro (robot description, xacro)
@@ -5,14 +5,14 @@
         <xacro:property name="head_offset" value="0.075" />
         <xacro:property name="neck_alignment" value="${PI/12}" />
-         <xacro:include filename="$(find talos_description)/urdf/head/head.transmission.xacro" />
+        <xacro:include filename="$(find talos_description)/urdf/head/head.transmission.xacro" />
 	<xacro:macro name="head" params="prefix parent *origin">
-                <!-- head which attackes to the pan unit, this is the tilt unit -->
-		<link name="${prefix}talos_head_link">
+              <!-- Stationary neck which attaches to the torso by fixed link -->
+              <link name="${prefix}talos_stationary_neck_link">
                   <mass value="${head_mass}"/>
                    <xacro:inertial_template mass="${head_mass}" length="${head_mass/12}" width="${head_mass/12}" height="${head_mass/12}"/>
 		  <visual>
-			<origin xyz="0 ${head_offset} 0" rpy="0 0 0"/>
+			<origin xyz="0 0 0" rpy="0 -${neck_alignment} 0"/>
 			<geometry>
-                           <mesh filename="package://talos_description/urdf/head/head.stl" scale="${scale} ${scale} ${scale}" />
+                           <mesh filename="package://talos_description/urdf/head/stationary_neck.stl" scale="${scale} ${scale} ${scale}" />
 			</geometry>
 			<material name="white"/>
@@ -21,10 +21,10 @@
                         <origin xyz="0 0 0" rpy="0 0 0"/>
 			<geometry>
-			  <mesh filename="package://talos_description/urdf/head/head.stl" scale="${scale} ${scale} ${scale}" />
+			  <mesh filename="package://talos_description/urdf/head/stationary_neck.stl" scale="${scale} ${scale} ${scale}" />
 			</geometry>
 		  </collision>
 		</link>
-              <!-- Neck which attaches to the torso and is the pan unit -->
-              <link name="${prefix}talos_neck_link">
+	      <!-- pan neck which attaches to the top of the stationary neck by continuous link -->
+              <link name="${prefix}talos_pan_neck_link">
                   <mass value="${head_mass}"/>
                    <xacro:inertial_template mass="${head_mass}" length="${head_mass/12}" width="${head_mass/12}" height="${head_mass/12}"/>
@@ -32,5 +32,5 @@
 			<origin xyz="0 0 0" rpy="0 -${neck_alignment} 0"/>
 			<geometry>
-                           <mesh filename="package://talos_description/urdf/head/neck.stl" scale="${scale} ${scale} ${scale}" />
+                           <mesh filename="package://talos_description/urdf/head/pan_neck.stl" scale="${scale} ${scale} ${scale}" />
 			</geometry>
 			<material name="white"/>
@@ -39,13 +39,31 @@
                         <origin xyz="0 0 0" rpy="0 0 0"/>
 			<geometry>
-			  <mesh filename="package://talos_description/urdf/head/neck.stl" scale="${scale} ${scale} ${scale}" />
+			  <mesh filename="package://talos_description/urdf/head/pan_neck.stl" scale="${scale} ${scale} ${scale}" />
 			</geometry>
 		  </collision>
 		</link>
-               <!-- Join head to neck (Tilt unit) -->
-               <joint name="${prefix}talos_head_joint" type="fixed">
+                 <!-- head which attackes to the pan unit, this is the tilt unit -->
+		<link name="${prefix}talos_tilt_head_link">
+                  <mass value="${head_mass}"/>
+                   <xacro:inertial_template mass="${head_mass}" length="${head_mass/12}" width="${head_mass/12}" height="${head_mass/12}"/>
+		  <visual>
+			<origin xyz="0 ${head_offset} 0" rpy="0 0 0"/>
+			<geometry>
+                           <mesh filename="package://talos_description/urdf/head/tilt_head.stl" scale="${scale} ${scale} ${scale}" />
+			</geometry>
+			<material name="white"/>
+		  </visual>
+		  <collision>
+                        <origin xyz="0 0 0" rpy="0 0 0"/>
+			<geometry>
+			  <mesh filename="package://talos_description/urdf/head/tilt_head.stl" scale="${scale} ${scale} ${scale}" />
+			</geometry>
+		  </collision>
+		</link>
+               <!-- Join tilt head to pan neck -->
+               <joint name="${prefix}talos_tilt_head_joint" type="revolute">
                    <origin xyz="0 0 0" rpy="0 0 0"/>
-                   <child link="${prefix}talos_head_link"/>
-                   <parent link="${prefix}talos_neck_link"/>
+                   <child link="${prefix}talos_tilt_head_link"/>
+                   <parent link="${prefix}talos_pan_neck_link"/>
                    <axis xyz="0 1 0" rpy="0 0 0"/>
                    <!-- <limit effort="100"
@@ -54,5 +72,5 @@
                                      friction="0.0" /> -->
                </joint>
-               <!-- Join neck to torso (Pan unit) -->
+               <!-- Join stationary neck to torso (fixed) -->
                <joint name="${prefix}talos_neck_joint" type="fixed">
                    <xacro:insert_block name="origin"/>
@@ -65,8 +83,22 @@
                                      friction="0.0" /> -->
                </joint>
-               <gazebo reference="${prefix}talos_head_link">
+               <!-- Join pan neck to stationary neck (rotational by 360) -->
+               <joint name="${prefix}talos_pan_neck_joint" type="continuous">
+                   <origin xyz="0 0 0" rpy="0 0 0"/>
+                   <child link="${prefix}talos_neck_link"/>
+                   <parent link="${prefix}talos_stationary_neck_link"/>
+                   <axis xyz="0 1 0" rpy="0 0 0"/>
+                   <!-- <limit effort="100"
+                          velocity="100" />
+                   <joint_properties damping="0.0"
+                                     friction="0.0" /> -->
+               </joint>
+               <gazebo reference="${prefix}talos_pan_neck_link">
                      <selfCollide>true</selfCollide>
 	       </gazebo>
-               <gazebo reference="${prefix}talos_neck_link">
+               <gazebo reference="${prefix}talos_tilt_head_link">
+                     <selfCollide>true</selfCollide>
+	       </gazebo>
+               <gazebo reference="${prefix}talos_stationary_neck_link">
                      <selfCollide>true</selfCollide>
 	       </gazebo>

Commit message: bugfixes

File: urdf/head/head.urdf.xacro (robot description, xacro)
@@ -14,5 +14,5 @@
 			<origin xyz="0 0 0" rpy="0 -${neck_alignment} 0"/>
 			<geometry>
-                           <mesh filename="package://talos_description/urdf/head/stationary_neck.stl" scale="${scale} ${scale} ${scale}" />
+                           <mesh filename="package://talos_description/meshes/head/stationary_neck.stl" scale="${scale} ${scale} ${scale}" />
 			</geometry>
 			<material name="white"/>
@@ -21,5 +21,5 @@
                         <origin xyz="0 0 0" rpy="0 0 0"/>
 			<geometry>
-			  <mesh filename="package://talos_description/urdf/head/stationary_neck.stl" scale="${scale} ${scale} ${scale}" />
+			  <mesh filename="package://talos_description/meshes/head/stationary_neck.stl" scale="${scale} ${scale} ${scale}" />
 			</geometry>
 		  </collision>
@@ -32,5 +32,5 @@
 			<origin xyz="0 0 0" rpy="0 -${neck_alignment} 0"/>
 			<geometry>
-                           <mesh filename="package://talos_description/urdf/head/pan_neck.stl" scale="${scale} ${scale} ${scale}" />
+                           <mesh filename="package://talos_description/meshes/head/pan_neck.stl" scale="${scale} ${scale} ${scale}" />
 			</geometry>
 			<material name="white"/>
@@ -39,5 +39,5 @@
                         <origin xyz="0 0 0" rpy="0 0 0"/>
 			<geometry>
-			  <mesh filename="package://talos_description/urdf/head/pan_neck.stl" scale="${scale} ${scale} ${scale}" />
+			  <mesh filename="package://talos_description/meshes/head/pan_neck.stl" scale="${scale} ${scale} ${scale}" />
 			</geometry>
 		  </collision>
@@ -50,5 +50,5 @@
 			<origin xyz="0 ${head_offset} 0" rpy="0 0 0"/>
 			<geometry>
-                           <mesh filename="package://talos_description/urdf/head/tilt_head.stl" scale="${scale} ${scale} ${scale}" />
+                           <mesh filename="package://talos_description/meshes/head/tilt_head.stl" scale="${scale} ${scale} ${scale}" />
 			</geometry>
 			<material name="white"/>
@@ -57,5 +57,5 @@
                         <origin xyz="0 0 0" rpy="0 0 0"/>
 			<geometry>
-			  <mesh filename="package://talos_description/urdf/head/tilt_head.stl" scale="${scale} ${scale} ${scale}" />
+			  <mesh filename="package://talos_description/meshes/head/tilt_head.stl" scale="${scale} ${scale} ${scale}" />
 			</geometry>
 		  </collision>
@@ -67,4 +67,5 @@
                    <parent link="${prefix}talos_pan_neck_link"/>
                    <axis xyz="0 1 0" rpy="0 0 0"/>
+                   <limit effort="1000.0" lower="0.0" upper="0.548" velocity="0.5"/>
                    <!-- <limit effort="100"
                           velocity="100" />
@@ -75,5 +76,5 @@
                <joint name="${prefix}talos_neck_joint" type="fixed">
                    <xacro:insert_block name="origin"/>
-                   <child link="${prefix}talos_neck_link"/>
+                   <child link="${prefix}talos_stationary_neck_link"/>
                    <parent link="${parent}"/>
                    <axis xyz="0 1 0" rpy="0 0 0"/>
@@ -86,5 +87,5 @@
                <joint name="${prefix}talos_pan_neck_joint" type="continuous">
                    <origin xyz="0 0 0" rpy="0 0 0"/>
-                   <child link="${prefix}talos_neck_link"/>
+                   <child link="${prefix}talos_pan_neck_link"/>
                    <parent link="${prefix}talos_stationary_neck_link"/>
                    <axis xyz="0 1 0" rpy="0 0 0"/>

File: urdf/sensors/sensors.urdf.xacro (robot description, xacro)
@@ -13,5 +13,5 @@
           <origin xyz="${hokuyo_x_offset} ${hokuyo_y_offset} ${hokuyo_z_offset}" rpy="0 0 -${PI/2}"/>
       </xacro:hokuyo>
-      <xacro:kinect parent="talos_head_link">
+      <xacro:kinect parent="talos_tilt_head_link">
           <origin xyz="${kinect_x_offset} ${kinect_y_offset} ${kinect_z_offset}" rpy="0 0 0"/>
       </xacro:kinect>

Commit message: Updated angle and position

File: urdf/head/head.urdf.xacro (robot description, xacro)
@@ -31,5 +31,5 @@
                    <xacro:inertial_template mass="${head_mass}" length="${head_mass/12}" width="${head_mass/12}" height="${head_mass/12}"/>
 		  <visual>
-			<origin xyz="0 0 0" rpy="0 ${PI/4} 0"/>
+			<origin xyz="0 0 0" rpy="0 ${5*PI/4} 0"/>
 			<geometry>
                            <mesh filename="package://talos_description/meshes/head/pan_neck.stl" scale="${scale} ${scale} ${scale}" />

Commit message: re-oriented pan_neck and tilt_head axes

File: urdf/head/head.urdf.xacro (robot description, xacro)
@@ -6,4 +6,6 @@
         <xacro:property name="neck_alignment" value="${PI/12}" />
         <xacro:property name="pan_rotation_alignment" value="${PI/8}"/>
+        <xacro:property name="pan_neck_to_tilt_head_z_offset" value="0.1638"/>
+        <xacro:property name="pan_neck_to_tilt_head_y_offset" value="0.05318"/>
         <xacro:include filename="$(find talos_description)/urdf/head/head.transmission.xacro" />
 	<xacro:macro name="head" params="prefix parent *origin">
@@ -31,5 +33,5 @@
                    <xacro:inertial_template mass="${head_mass}" length="${head_mass/12}" width="${head_mass/12}" height="${head_mass/12}"/>
 		  <visual>
-			<origin xyz="0 0 0" rpy="0 ${5*PI/4} 0"/>
+			<origin xyz="0 0 0" rpy="0 0 0"/>
 			<geometry>
                            <mesh filename="package://talos_description/meshes/head/pan_neck.stl" scale="${scale} ${scale} ${scale}" />
@@ -44,10 +46,10 @@
 		  </collision>
 		</link>
-                 <!-- head which attackes to the pan unit, this is the tilt unit -->
+                 <!-- head which attaches to the pan unit, this is the tilt unit -->
 		<link name="${prefix}talos_tilt_head_link">
                   <mass value="${head_mass}"/>
                    <xacro:inertial_template mass="${head_mass}" length="${head_mass/12}" width="${head_mass/12}" height="${head_mass/12}"/>
 		  <visual>
-			<origin xyz="0 ${head_offset} 0" rpy="0 0 0"/>
+			<origin xyz="0 0 0" rpy="0 0 0"/>
 			<geometry>
                            <mesh filename="package://talos_description/meshes/head/tilt_head.stl" scale="${scale} ${scale} ${scale}" />
@@ -64,5 +66,5 @@
                <!-- Join tilt head to pan neck -->
                <joint name="${prefix}talos_tilt_head_joint" type="revolute">
-                   <origin xyz="0 0 0" rpy="0 0 0"/>
+                   <origin xyz="0 ${pan_neck_to_tilt_head_y_offset} ${pan_neck_to_tilt_head_z_offset}" rpy="0 0 0"/>
                    <child link="${prefix}talos_tilt_head_link"/>
                    <parent link="${prefix}talos_pan_neck_link"/>
@@ -87,5 +89,5 @@
                <!-- Join pan neck to stationary neck (rotational by 360) -->
                <joint name="${prefix}talos_pan_neck_joint" type="continuous">
-                   <origin xyz="0 0 0" rpy="0 0 0"/>
+                   <origin xyz="0 0 ${head_offset}" rpy="0 0 0"/>
                    <child link="${prefix}talos_pan_neck_link"/>
                    <parent link="${prefix}talos_stationary_neck_link"/>

Commit message: edited tilt_head axis of motion

File: urdf/head/head.urdf.xacro (robot description, xacro)
@@ -69,6 +69,7 @@
                    <child link="${prefix}talos_tilt_head_link"/>
                    <parent link="${prefix}talos_pan_neck_link"/>
-                   <axis xyz="0 1 0" rpy="0 0 0"/>
-                   <limit effort="1000.0" lower="0.0" upper="0.548" velocity="0.5"/>
+                   <axis xyz="1 0 0" rpy="0 0 0"/>
+		   <limit effort="1000.0" lower="-0.35" upper="0.19" velocity="0.5"/>
+                   <!-- <limit effort="1000.0" lower="0.0" upper="0.548" velocity="0.5"/>-->
                    <!-- <limit effort="100"
                           velocity="100" />
